Commit message: Removed dual camera support and physical hardware nodes, updated README.md.

File: lunabot_simulation/urdf/robot/rectangle_bot.xacro (robot description, xacro)
@@ -1,4 +1,4 @@
 <?xml version="1.0"?>
-<robot name="square_bot"
+<robot name="rectangle_bot"
   xmlns:xacro="http://www.ros.org/wiki/xacro">
   <material name="light_grey">
@@ -15,7 +15,12 @@
   </material>
   <link name="base_link">
-    <visual>
-      <geometry>
-        <mesh filename="file:///$(find lunabot_simulation)/models/square_bot/square_bot_body.stl" />
+    <inertial>
+      <mass value="25.0" />
+      <origin xyz="0 0 0.085" />
+      <inertia ixx="1.3669" ixy="0.0" ixz="0.0" iyy="3.3602" iyz="0.0" izz="4.7271" />
+    </inertial>
+    <visual>
+      <geometry>
+        <mesh filename="file:///$(find lunabot_simulation)/models/rectangle_bot/rectangle_bot.stl" />
       </geometry>
       <origin xyz="0 0 0.1625" rpy="0 0 0" />
@@ -24,13 +29,8 @@
     <collision>
       <geometry>
-        <mesh filename="file:///$(find lunabot_simulation)/models/square_bot/square_bot_body.stl" />
-      </geometry>
-      <origin xyz="0 0 0.1625" rpy="0 0 0" />
-    </collision>
-    <inertial>
-      <mass value="25.0" />
-      <origin xyz="0 0 0.1625" />
-      <inertia ixx="1.3669" ixy="0.0" ixz="0.0" iyy="3.3602" iyz="0.0" izz="4.7271" />
-    </inertial>
+        <mesh filename="file:///$(find lunabot_simulation)/models/rectangle_bot/rectangle_bot.stl" />
+      </geometry>
+      <origin xyz="0 0 0.085" rpy="0 0 0" />
+    </collision>
   </link>
   <link name="lidar_link">
@@ -52,5 +52,5 @@
     <visual>
       <geometry>
-        <mesh filename="file:///$(find lunabot_simulation)/models/square_bot/square_bot_blade.stl" />
+        <mesh filename="file:///$(find lunabot_simulation)/models/rectangle_bot/rectangle_bot_blade.stl" />
       </geometry>
       <origin xyz="0 0 0" rpy="0 0 0" />
@@ -59,5 +59,5 @@
     <collision>
       <geometry>
-        <mesh filename="file:///$(find lunabot_simulation)/models/square_bot/square_bot_blade.stl" />
+        <mesh filename="file:///$(find lunabot_simulation)/models/rectangle_bot/rectangle_bot_blade.stl" />
       </geometry>
       <origin xyz="0 0 0" rpy="0 0 0" />
@@ -69,20 +69,4 @@
     </inertial>
   </link>
-  <link name="d455_link">
-    <visual>
-      <geometry>
-        <mesh filename="file:///$(find lunabot_simulation)/models/d455_camera/d455_camera.stl" />
-      </geometry>
-      <origin xyz="0 0 0" rpy="0 0 0" />
-      <material name="camera_grey" />
-    </visual>
-    <collision>
-      <geometry>
-        <mesh filename="file:///$(find lunabot_simulation)/models/d455_camera/d455_camera.stl" />
-      </geometry>
-      <origin xyz="0 0 0" rpy="0 0 0" />
-    </collision>
-  </link>
-  <link name="d455_optical_link"></link>
   <link name="d456_link">
     <visual>
@@ -103,4 +87,11 @@
   <link name="imu_link"></link>
   <link name="front_right_wheel_link">
+    <visual>
+      <geometry>
+        <mesh filename="file:///$(find lunabot_simulation)/models/wheel/wheel.stl" />
+      </geometry>
+      <origin xyz="0 0 0" rpy="1.5708 0 0" />
+      <material name="black" />
+    </visual>
     <inertial>
       <mass value="2.27" />
@@ -110,5 +101,5 @@
     <collision>
       <geometry>
-        <cylinder length="0.127" radius="0.1016" />
+        <mesh filename="file:///$(find lunabot_simulation)/models/wheel/wheel.stl" />
       </geometry>
       <origin xyz="0 0 0" rpy="1.5708 0 0" />
@@ -116,4 +107,11 @@
   </link>
   <link name="front_left_wheel_link">
+    <visual>
+      <geometry>
+        <mesh filename="file:///$(find lunabot_simulation)/models/wheel/wheel.stl" />
+      </geometry>
+      <origin xyz="0 0 0" rpy="-1.5708 0 0" />
+      <material name="black" />
+    </visual>
     <inertial>
       <mass value="2.27" />
@@ -123,5 +121,5 @@
     <collision>
       <geometry>
-        <cylinder length="0.127" radius="0.1016" />
+        <mesh filename="file:///$(find lunabot_simulation)/models/wheel/wheel.stl" />
       </geometry>
       <origin xyz="0 0 0" rpy="-1.5708 0 0" />
@@ -129,4 +127,11 @@
   </link>
   <link name="rear_right_wheel_link">
+    <visual>
+      <geometry>
+        <mesh filename="file:///$(find lunabot_simulation)/models/wheel/wheel.stl" />
+      </geometry>
+      <origin xyz="0 0 0" rpy="1.5708 0 0" />
+      <material name="black" />
+    </visual>
     <inertial>
       <mass value="2.27" />
@@ -136,5 +141,5 @@
     <collision>
       <geometry>
-        <cylinder length="0.127" radius="0.1016" />
+        <mesh filename="file:///$(find lunabot_simulation)/models/wheel/wheel.stl" />
       </geometry>
       <origin xyz="0 0 0" rpy="1.5708 0 0" />
@@ -142,4 +147,11 @@
   </link>
   <link name="rear_left_wheel_link">
+    <visual>
+      <geometry>
+        <mesh filename="file:///$(find lunabot_simulation)/models/wheel/wheel.stl" />
+      </geometry>
+      <origin xyz="0 0 0" rpy="-1.5708 0 0" />
+      <material name="black" />
+    </visual>
     <inertial>
       <mass value="2.27" />
@@ -149,5 +161,5 @@
     <collision>
       <geometry>
-        <cylinder length="0.127" radius="0.1016" />
+        <mesh filename="file:///$(find lunabot_simulation)/models/wheel/wheel.stl" />
       </geometry>
       <origin xyz="0 0 0" rpy="-1.5708 0 0" />
@@ -157,11 +169,11 @@
     <parent link="base_link" />
     <child link="rear_right_wheel_link" />
-    <origin xyz="-0.235 -0.25 0.08" rpy="0 0 0" />
+    <origin xyz="-0.19 -0.25 0.085" rpy="0 0 0" />
     <axis xyz="0 1 0" />
   </joint>
   <joint name="base_rear_left_wheel_joint" type="continuous">
-    <parent link="base_link" />0 <child link="rear_left_wheel_link" />
-    <origin xyz="-0.235 0.25 0.08"
-      rpy="0 0 0" />
+    <parent link="base_link" />
+    <child link="rear_left_wheel_link" />
+    <origin xyz="-0.19 0.25 0.085" rpy="0 0 0" />
     <axis xyz="0 1 0" />
   </joint>
@@ -169,5 +181,5 @@
     <parent link="base_link" />
     <child link="front_right_wheel_link" />
-    <origin xyz="0.215 -0.25 0.08" rpy="0 0 0" />
+    <origin xyz="0.28 -0.25 0.085" rpy="0 0 0" />
     <axis xyz="0 1 0" />
   </joint>
@@ -175,5 +187,5 @@
     <parent link="base_link" />
     <child link="front_left_wheel_link" />
-    <origin xyz="0.215 0.25 0.08" rpy="0 0 0" />
+    <origin xyz="0.28 0.25 0.085" rpy="0 0 0" />
     <axis xyz="0 1 0" />
   </joint>
@@ -181,28 +193,18 @@
     <parent link="base_link" />
     <child link="lidar_link" />
-    <origin xyz="-0.013 0 0.56" rpy="0 0 0" />
+    <origin xyz="-0.0925 0 0.405" rpy="0 0 0" />
   </joint>
   <joint name="base_blade_joint" type="revolute">
     <parent link="base_link" />
     <child link="blade_link" />
-    <origin xyz="-0.4 0.0 0.08" rpy="0 -0.4 3.14" />
+    <origin xyz="-0.55 0.0 0.14" rpy="0 -0.4 3.14" />
     <axis xyz="0 1 0" />
     <limit effort="100" velocity="1.0" lower="-0.75" upper="0.75" />
     <dynamics damping="0.0" friction="0.0" />
   </joint>
-  <joint name="base_d455_joint" type="fixed">
-    <parent link="base_link" />
-    <child link="d455_link" />
-    <origin xyz="-0.038 0 0.5" rpy="0 0 3.14" />
-  </joint>
-  <joint name="d455_optical_joint" type="fixed">
-    <parent link="d455_link" />
-    <child link="d455_optical_link" />
-    <origin xyz="0 0 0" rpy="-1.5708 0 -1.5708" />
-  </joint>
   <joint name="base_d456_joint" type="fixed">
     <parent link="base_link" />
     <child link="d456_link" />
-    <origin xyz="0.025 0 0.5" rpy="0 0.523599 0" />
+    <origin xyz="-0.05 0 0.355" rpy="0 0.523599 0" />
   </joint>
   <joint name="d456_optical_joint" type="fixed">
@@ -219,9 +221,12 @@
     <material>Gazebo/Grey</material>
   </gazebo>
+  <gazebo reference="ebox_link">
+    <material>Gazebo/White</material>
+  </gazebo>
   <gazebo reference="blade_link">
     <material>Gazebo/Grey</material>
   </gazebo>
   <gazebo reference="front_right_wheel_link">
-    <material>Gazebo/Grey</material>
+    <material>Gazebo/DarkGrey</material>
     <mu>1.0</mu>
     <mu2>1.0</mu2>
@@ -238,5 +243,5 @@
   </gazebo>
   <gazebo reference="front_left_wheel_link">
-    <material>Gazebo/Grey</material>
+    <material>Gazebo/DarkGrey</material>
     <mu>1.0</mu>
     <mu2>1.0</mu2>
@@ -253,5 +258,5 @@
   </gazebo>
   <gazebo reference="rear_right_wheel_link">
-    <material>Gazebo/Grey</material>
+    <material>Gazebo/DarkGrey</material>
     <mu>1.0</mu>
     <mu2>1.0</mu2>
@@ -268,5 +273,5 @@
   </gazebo>
   <gazebo reference="rear_left_wheel_link">
-    <material>Gazebo/Grey</material>
+    <material>Gazebo/DarkGrey</material>
     <mu>1.0</mu>
     <mu2>1.0</mu2>
@@ -281,42 +286,4 @@
       </contact>
     </surface>
-  </gazebo>
-  <gazebo reference="d455_link">
-    <sensor type="depth" name="d455">
-      <pose>0 0 0 0 0 0</pose>
-      <update_rate>60.0</update_rate>
-      <visualize>true</visualize>
-      <camera>
-        <horizontal_fov>1.540</horizontal_fov>
-        <image>
-          <width>640</width>
-          <height>360</height>
-          <format>R8G8B8</format>
-        </image>
-        <distortion>
-          <k1>-0.06792929080519726</k1>
-          <k2>0.08058277259698843</k2>
-          <k3>-0.04417756393089296</k3>
-          <p1>-0.001690544521662593</p1>
-          <p2>-0.0008235437909836152</p2>
-        </distortion>
-        <clip>
-          <near>0.05</near>
-          <far>10.0</far>
-        </clip>
-      </camera>
-      <plugin name="camera1_controller" filename="libgazebo_ros_camera.so">
-        <ros>
-          <remapping>/d455/image_raw:=/d455/color/image_raw</remapping>
-          <remapping>/d455/points:=/d455/color/points</remapping>
-          <remapping>/d455/camera_info:=/d455/color/camera_info</remapping>
-          <remapping>/d455/depth/image_raw:=/d455/depth/image_rect_raw</remapping>
-        </ros>
-        <frame_name>d455_optical_link</frame_name>
-        <publish_tf>false</publish_tf>
-        <publish_point_cloud>true</publish_point_cloud>
-      </plugin>
-    </sensor>
-    <material>Gazebo/Grey</material>
   </gazebo>
   <gazebo reference="d456_link">
@@ -344,5 +311,5 @@
         </clip>
       </camera>
-      <plugin name="camera2_controller" filename="libgazebo_ros_camera.so">
+      <plugin name="camera_controller" filename="libgazebo_ros_camera.so">
         <ros>
           <remapping>/d456/image_raw:=/d456/color/image_raw</remapping>

File: lunabot_simulation/urdf/robot/square_bot.xacro (robot description, xacro)
@@ -1,4 +1,4 @@
 <?xml version="1.0"?>
-<robot name="rectangle_bot"
+<robot name="square_bot"
   xmlns:xacro="http://www.ros.org/wiki/xacro">
   <material name="light_grey">
@@ -15,12 +15,7 @@
   </material>
   <link name="base_link">
-    <inertial>
-      <mass value="25.0" />
-      <origin xyz="0 0 0.085" />
-      <inertia ixx="1.3669" ixy="0.0" ixz="0.0" iyy="3.3602" iyz="0.0" izz="4.7271" />
-    </inertial>
     <visual>
       <geometry>
-        <mesh filename="file:///$(find lunabot_simulation)/models/rectangle_bot/rectangle_bot.stl" />
+        <mesh filename="file:///$(find lunabot_simulation)/models/square_bot/square_bot_body.stl" />
       </geometry>
       <origin xyz="0 0 0.1625" rpy="0 0 0" />
@@ -29,8 +24,13 @@
     <collision>
       <geometry>
-        <mesh filename="file:///$(find lunabot_simulation)/models/rectangle_bot/rectangle_bot.stl" />
-      </geometry>
-      <origin xyz="0 0 0.085" rpy="0 0 0" />
-    </collision>
+        <mesh filename="file:///$(find lunabot_simulation)/models/square_bot/square_bot_body.stl" />
+      </geometry>
+      <origin xyz="0 0 0.1625" rpy="0 0 0" />
+    </collision>
+    <inertial>
+      <mass value="25.0" />
+      <origin xyz="0 0 0.1625" />
+      <inertia ixx="1.3669" ixy="0.0" ixz="0.0" iyy="3.3602" iyz="0.0" izz="4.7271" />
+    </inertial>
   </link>
   <link name="lidar_link">
@@ -52,5 +52,5 @@
     <visual>
       <geometry>
-        <mesh filename="file:///$(find lunabot_simulation)/models/rectangle_bot/rectangle_bot_blade.stl" />
+        <mesh filename="file:///$(find lunabot_simulation)/models/square_bot/square_bot_blade.stl" />
       </geometry>
       <origin xyz="0 0 0" rpy="0 0 0" />
@@ -59,5 +59,5 @@
     <collision>
       <geometry>
-        <mesh filename="file:///$(find lunabot_simulation)/models/rectangle_bot/rectangle_bot_blade.stl" />
+        <mesh filename="file:///$(find lunabot_simulation)/models/square_bot/square_bot_blade.stl" />
       </geometry>
       <origin xyz="0 0 0" rpy="0 0 0" />
@@ -69,8 +69,8 @@
     </inertial>
   </link>
-  <link name="d455_link">
+  <link name="d456_link">
     <visual>
       <geometry>
-        <mesh filename="file:///$(find lunabot_simulation)/models/d455_camera/d455_camera.stl" />
+        <mesh filename="file:///$(find lunabot_simulation)/models/d456_camera/d456_camera.stl" />
       </geometry>
       <origin xyz="0 0 0" rpy="0 0 0" />
@@ -79,20 +79,4 @@
     <collision>
       <geometry>
-        <mesh filename="file:///$(find lunabot_simulation)/models/d455_camera/d455_camera.stl" />
-      </geometry>
-      <origin xyz="0 0 0" rpy="0 0 0" />
-    </collision>
-  </link>
-  <link name="d455_optical_link"></link>
-  <link name="d456_link">
-    <visual>
-      <geometry>
-        <mesh filename="file:///$(find lunabot_simulation)/models/d456_camera/d456_camera.stl" />
-      </geometry>
-      <origin xyz="0 0 0" rpy="0 0 0" />
-      <material name="camera_grey" />
-    </visual>
-    <collision>
-      <geometry>
         <mesh filename="file:///$(find lunabot_simulation)/models/d456_camera/d456_camera.stl" />
       </geometry>
@@ -103,11 +87,4 @@
   <link name="imu_link"></link>
   <link name="front_right_wheel_link">
-    <visual>
-      <geometry>
-        <mesh filename="file:///$(find lunabot_simulation)/models/wheel/wheel.stl" />
-      </geometry>
-      <origin xyz="0 0 0" rpy="1.5708 0 0" />
-      <material name="black" />
-    </visual>
     <inertial>
       <mass value="2.27" />
@@ -117,5 +94,5 @@
     <collision>
       <geometry>
-        <mesh filename="file:///$(find lunabot_simulation)/models/wheel/wheel.stl" />
+        <cylinder length="0.127" radius="0.1016" />
       </geometry>
       <origin xyz="0 0 0" rpy="1.5708 0 0" />
@@ -123,11 +100,4 @@
   </link>
   <link name="front_left_wheel_link">
-    <visual>
-      <geometry>
-        <mesh filename="file:///$(find lunabot_simulation)/models/wheel/wheel.stl" />
-      </geometry>
-      <origin xyz="0 0 0" rpy="-1.5708 0 0" />
-      <material name="black" />
-    </visual>
     <inertial>
       <mass value="2.27" />
@@ -137,5 +107,5 @@
     <collision>
       <geometry>
-        <mesh filename="file:///$(find lunabot_simulation)/models/wheel/wheel.stl" />
+        <cylinder length="0.127" radius="0.1016" />
       </geometry>
       <origin xyz="0 0 0" rpy="-1.5708 0 0" />
@@ -143,11 +113,4 @@
   </link>
   <link name="rear_right_wheel_link">
-    <visual>
-      <geometry>
-        <mesh filename="file:///$(find lunabot_simulation)/models/wheel/wheel.stl" />
-      </geometry>
-      <origin xyz="0 0 0" rpy="1.5708 0 0" />
-      <material name="black" />
-    </visual>
     <inertial>
       <mass value="2.27" />
@@ -157,5 +120,5 @@
     <collision>
       <geometry>
-        <mesh filename="file:///$(find lunabot_simulation)/models/wheel/wheel.stl" />
+        <cylinder length="0.127" radius="0.1016" />
       </geometry>
       <origin xyz="0 0 0" rpy="1.5708 0 0" />
@@ -163,11 +126,4 @@
   </link>
   <link name="rear_left_wheel_link">
-    <visual>
-      <geometry>
-        <mesh filename="file:///$(find lunabot_simulation)/models/wheel/wheel.stl" />
-      </geometry>
-      <origin xyz="0 0 0" rpy="-1.5708 0 0" />
-      <material name="black" />
-    </visual>
     <inertial>
       <mass value="2.27" />
@@ -177,5 +133,5 @@
     <collision>
       <geometry>
-        <mesh filename="file:///$(find lunabot_simulation)/models/wheel/wheel.stl" />
+        <cylinder length="0.127" radius="0.1016" />
       </geometry>
       <origin xyz="0 0 0" rpy="-1.5708 0 0" />
@@ -185,11 +141,11 @@
     <parent link="base_link" />
     <child link="rear_right_wheel_link" />
-    <origin xyz="-0.19 -0.25 0.085" rpy="0 0 0" />
+    <origin xyz="-0.235 -0.25 0.08" rpy="0 0 0" />
     <axis xyz="0 1 0" />
   </joint>
   <joint name="base_rear_left_wheel_joint" type="continuous">
-    <parent link="base_link" />
-    <child link="rear_left_wheel_link" />
-    <origin xyz="-0.19 0.25 0.085" rpy="0 0 0" />
+    <parent link="base_link" />0 <child link="rear_left_wheel_link" />
+    <origin xyz="-0.235 0.25 0.08"
+      rpy="0 0 0" />
     <axis xyz="0 1 0" />
   </joint>
@@ -197,5 +153,5 @@
     <parent link="base_link" />
     <child link="front_right_wheel_link" />
-    <origin xyz="0.28 -0.25 0.085" rpy="0 0 0" />
+    <origin xyz="0.215 -0.25 0.08" rpy="0 0 0" />
     <axis xyz="0 1 0" />
   </joint>
@@ -203,5 +159,5 @@
     <parent link="base_link" />
     <child link="front_left_wheel_link" />
-    <origin xyz="0.28 0.25 0.085" rpy="0 0 0" />
+    <origin xyz="0.215 0.25 0.08" rpy="0 0 0" />
     <axis xyz="0 1 0" />
   </joint>
@@ -209,28 +165,18 @@
     <parent link="base_link" />
     <child link="lidar_link" />
-    <origin xyz="-0.0925 0 0.405" rpy="0 0 0" />
+    <origin xyz="-0.013 0 0.56" rpy="0 0 0" />
   </joint>
   <joint name="base_blade_joint" type="revolute">
     <parent link="base_link" />
     <child link="blade_link" />
-    <origin xyz="-0.55 0.0 0.14" rpy="0 -0.4 3.14" />
+    <origin xyz="-0.4 0.0 0.08" rpy="0 -0.4 3.14" />
     <axis xyz="0 1 0" />
     <limit effort="100" velocity="1.0" lower="-0.75" upper="0.75" />
     <dynamics damping="0.0" friction="0.0" />
   </joint>
-  <joint name="base_d455_joint" type="fixed">
-    <parent link="base_link" />
-    <child link="d455_link" />
-    <origin xyz="-0.12 0 0.355" rpy="0 0 3.14" />
-  </joint>
-  <joint name="d455_optical_joint" type="fixed">
-    <parent link="d455_link" />
-    <child link="d455_optical_link" />
-    <origin xyz="0 0 0" rpy="-1.5708 0 -1.5708" />
-  </joint>
   <joint name="base_d456_joint" type="fixed">
     <parent link="base_link" />
     <child link="d456_link" />
-    <origin xyz="-0.05 0 0.355" rpy="0 0.523599 0" />
+    <origin xyz="0.025 0 0.5" rpy="0 0.523599 0" />
   </joint>
   <joint name="d456_optical_joint" type="fixed">
@@ -247,12 +193,9 @@
     <material>Gazebo/Grey</material>
   </gazebo>
-  <gazebo reference="ebox_link">
-    <material>Gazebo/White</material>
-  </gazebo>
   <gazebo reference="blade_link">
     <material>Gazebo/Grey</material>
   </gazebo>
   <gazebo reference="front_right_wheel_link">
-    <material>Gazebo/DarkGrey</material>
+    <material>Gazebo/Grey</material>
     <mu>1.0</mu>
     <mu2>1.0</mu2>
@@ -269,5 +212,5 @@
   </gazebo>
   <gazebo reference="front_left_wheel_link">
-    <material>Gazebo/DarkGrey</material>
+    <material>Gazebo/Grey</material>
     <mu>1.0</mu>
     <mu2>1.0</mu2>
@@ -284,5 +227,5 @@
   </gazebo>
   <gazebo reference="rear_right_wheel_link">
-    <material>Gazebo/DarkGrey</material>
+    <material>Gazebo/Grey</material>
     <mu>1.0</mu>
     <mu2>1.0</mu2>
@@ -299,5 +242,5 @@
   </gazebo>
   <gazebo reference="rear_left_wheel_link">
-    <material>Gazebo/DarkGrey</material>
+    <material>Gazebo/Grey</material>
     <mu>1.0</mu>
     <mu2>1.0</mu2>
@@ -312,42 +255,4 @@
       </contact>
     </surface>
-  </gazebo>
-  <gazebo reference="d455_link">
-    <sensor type="depth" name="d455">
-      <pose>0 0 0 0 0 0</pose>
-      <update_rate>60.0</update_rate>
-      <visualize>true</visualize>
-      <camera>
-        <horizontal_fov>1.540</horizontal_fov>
-        <image>
-          <width>640</width>
-          <height>360</height>
-          <format>R8G8B8</format>
-        </image>
-        <distortion>
-          <k1>-0.06792929080519726</k1>
-          <k2>0.08058277259698843</k2>
-          <k3>-0.04417756393089296</k3>
-          <p1>-0.001690544521662593</p1>
-          <p2>-0.0008235437909836152</p2>
-        </distortion>
-        <clip>
-          <near>0.05</near>
-          <far>10.0</far>
-        </clip>
-      </camera>
-      <plugin name="camera1_controller" filename="libgazebo_ros_camera.so">
-        <ros>
-          <remapping>/d455/image_raw:=/d455/color/image_raw</remapping>
-          <remapping>/d455/points:=/d455/color/points</remapping>
-          <remapping>/d455/camera_info:=/d455/color/camera_info</remapping>
-          <remapping>/d455/depth/image_raw:=/d455/depth/image_rect_raw</remapping>
-        </ros>
-        <frame_name>d455_optical_link</frame_name>
-        <publish_tf>false</publish_tf>
-        <publish_point_cloud>true</publish_point_cloud>
-      </plugin>
-    </sensor>
-    <material>Gazebo/Grey</material>
   </gazebo>
   <gazebo reference="d456_link">
@@ -375,5 +280,5 @@
         </clip>
       </camera>
-      <plugin name="camera2_controller" filename="libgazebo_ros_camera.so">
+      <plugin name="camera_controller" filename="libgazebo_ros_camera.so">
         <ros>
           <remapping>/d456/image_raw:=/d456/color/image_raw</remapping>
