Commit message: Removed dual camera support and physical hardware nodes, updated README.md.

File: lunabot_simulation/urdf/robot/trencher_bot.xacro (robot description, xacro)
@@ -1,4 +1,4 @@
 <?xml version="1.0"?>
-<robot name="realistic_rectangle_bot"
+<robot name="trencher_bot"
   xmlns:xacro="http://www.ros.org/wiki/xacro">
   <material name="light_grey">
@@ -17,14 +17,13 @@
     <visual>
       <geometry>
-        <mesh filename="file:///$(find lunabot_simulation)/models/rectangle_bot/rectangle_bot_body.dae" />
-      </geometry>
-      <origin xyz="0 0 0.1625" rpy="0 0 0" />
-      <material name="light_grey" />
+        <mesh filename="file:///$(find lunabot_simulation)/models/trencher_bot/trencher_bot.dae" />
+      </geometry>
+      <origin xyz="0 0.0125 0.3" rpy="0 0 0" />
     </visual>
     <collision>
       <geometry>
-        <mesh filename="file:///$(find lunabot_simulation)/models/rectangle_bot/rectangle_bot_body.stl" />
-      </geometry>
-      <origin xyz="0 0 0.085" rpy="0 0 0" />
+        <mesh filename="file:///$(find lunabot_simulation)/models/trencher_bot/trencher_bot.stl" />
+      </geometry>
+      <origin xyz="0 0.0125 0.3" rpy="0 0 0" />
     </collision>
     <inertial>
@@ -49,28 +48,8 @@
     </collision>
   </link>
-  <link name="blade_link">
+  <link name="d456_link">
     <visual>
       <geometry>
-        <mesh filename="file:///$(find lunabot_simulation)/models/rectangle_bot/rectangle_bot_blade.dae" />
-      </geometry>
-      <origin xyz="0 0 0" rpy="0 0 0" />
-      <material name="light_grey" />
-    </visual>
-    <collision>
-      <geometry>
-        <mesh filename="file:///$(find lunabot_simulation)/models/rectangle_bot/rectangle_bot_blade.stl" />
-      </geometry>
-      <origin xyz="0 0 0" rpy="0 0 0" />
-    </collision>
-    <inertial>
-      <mass value="5.0" />
-      <origin xyz="0 0 0" />
-      <inertia ixx="0.0833" ixy="0.0" ixz="0.0" iyy="0.1667" iyz="0.0" izz="0.2333" />
-    </inertial>
-  </link>
-  <link name="d455_link">
-    <visual>
-      <geometry>
-        <mesh filename="file:///$(find lunabot_simulation)/models/d455_camera/d455_camera.stl" />
+        <mesh filename="file:///$(find lunabot_simulation)/models/d456_camera/d456_camera.stl" />
       </geometry>
       <origin xyz="0 0 0" rpy="0 0 0" />
@@ -79,20 +58,4 @@
     <collision>
       <geometry>
-        <mesh filename="file:///$(find lunabot_simulation)/models/d455_camera/d455_camera.stl" />
-      </geometry>
-      <origin xyz="0 0 0" rpy="0 0 0" />
-    </collision>
-  </link>
-  <link name="d455_optical_link"></link>
-  <link name="d456_link">
-    <visual>
-      <geometry>
-        <mesh filename="file:///$(find lunabot_simulation)/models/d456_camera/d456_camera.stl" />
-      </geometry>
-      <origin xyz="0 0 0" rpy="0 0 0" />
-      <material name="camera_grey" />
-    </visual>
-    <collision>
-      <geometry>
         <mesh filename="file:///$(find lunabot_simulation)/models/d456_camera/d456_camera.stl" />
       </geometry>
@@ -103,11 +66,4 @@
   <link name="imu_link"></link>
   <link name="front_right_wheel_link">
-    <visual>
-      <geometry>
-        <mesh filename="file:///$(find lunabot_simulation)/models/wheel/wheel.stl" />
-      </geometry>
-      <origin xyz="0 0 0" rpy="1.5708 0 0" />
-      <material name="black" />
-    </visual>
     <inertial>
       <mass value="2.27" />
@@ -117,5 +73,5 @@
     <collision>
       <geometry>
-        <mesh filename="file:///$(find lunabot_simulation)/models/wheel/wheel.stl" />
+        <cylinder length="0.127" radius="0.14" />
       </geometry>
       <origin xyz="0 0 0" rpy="1.5708 0 0" />
@@ -123,11 +79,4 @@
   </link>
   <link name="front_left_wheel_link">
-    <visual>
-      <geometry>
-        <mesh filename="file:///$(find lunabot_simulation)/models/wheel/wheel.stl" />
-      </geometry>
-      <origin xyz="0 0 0" rpy="-1.5708 0 0" />
-      <material name="black" />
-    </visual>
     <inertial>
       <mass value="2.27" />
@@ -137,5 +86,5 @@
     <collision>
       <geometry>
-        <mesh filename="file:///$(find lunabot_simulation)/models/wheel/wheel.stl" />
+        <cylinder length="0.127" radius="0.14" />
       </geometry>
       <origin xyz="0 0 0" rpy="-1.5708 0 0" />
@@ -143,11 +92,4 @@
   </link>
   <link name="rear_right_wheel_link">
-    <visual>
-      <geometry>
-        <mesh filename="file:///$(find lunabot_simulation)/models/wheel/wheel.stl" />
-      </geometry>
-      <origin xyz="0 0 0" rpy="1.5708 0 0" />
-      <material name="black" />
-    </visual>
     <inertial>
       <mass value="2.27" />
@@ -157,5 +99,5 @@
     <collision>
       <geometry>
-        <mesh filename="file:///$(find lunabot_simulation)/models/wheel/wheel.stl" />
+        <cylinder length="0.127" radius="0.14" />
       </geometry>
       <origin xyz="0 0 0" rpy="1.5708 0 0" />
@@ -163,11 +105,4 @@
   </link>
   <link name="rear_left_wheel_link">
-    <visual>
-      <geometry>
-        <mesh filename="file:///$(find lunabot_simulation)/models/wheel/wheel.stl" />
-      </geometry>
-      <origin xyz="0 0 0" rpy="-1.5708 0 0" />
-      <material name="black" />
-    </visual>
     <inertial>
       <mass value="2.27" />
@@ -177,5 +112,5 @@
     <collision>
       <geometry>
-        <mesh filename="file:///$(find lunabot_simulation)/models/wheel/wheel.stl" />
+        <cylinder length="0.127" radius="0.14" />
       </geometry>
       <origin xyz="0 0 0" rpy="-1.5708 0 0" />
@@ -185,5 +120,5 @@
     <parent link="base_link" />
     <child link="rear_right_wheel_link" />
-    <origin xyz="-0.305 -0.25 0.105" rpy="0 0 0" />
+    <origin xyz="-0.305 -0.25 0.08" rpy="0 0 0" />
     <axis xyz="0 1 0" />
   </joint>
@@ -191,5 +126,5 @@
     <parent link="base_link" />
     <child link="rear_left_wheel_link" />
-    <origin xyz="-0.305 0.25 0.105" rpy="0 0 0" />
+    <origin xyz="-0.305 0.25 0.08" rpy="0 0 0" />
     <axis xyz="0 1 0" />
   </joint>
@@ -197,5 +132,5 @@
     <parent link="base_link" />
     <child link="front_right_wheel_link" />
-    <origin xyz="0.1515 -0.25 0.105" rpy="0 0 0" />
+    <origin xyz="0.1515 -0.25 0.08" rpy="0 0 0" />
     <axis xyz="0 1 0" />
   </joint>
@@ -203,5 +138,5 @@
     <parent link="base_link" />
     <child link="front_left_wheel_link" />
-    <origin xyz="0.1515 0.25 0.105" rpy="0 0 0" />
+    <origin xyz="0.1515 0.25 0.08" rpy="0 0 0" />
     <axis xyz="0 1 0" />
   </joint>
@@ -209,28 +144,10 @@
     <parent link="base_link" />
     <child link="lidar_link" />
-    <origin xyz="-0.075 0 0.575" rpy="0 0 0" />
-  </joint>
-  <joint name="base_blade_joint" type="revolute">
-    <parent link="base_link" />
-    <child link="blade_link" />
-    <origin xyz="-0.54 0.0 0.12" rpy="0 -0.6 3.14" />
-    <axis xyz="0 1 0" />
-    <limit effort="100" velocity="1.0" lower="-0.75" upper="0.75" />
-    <dynamics damping="0.0" friction="0.0" />
-  </joint>
-  <joint name="base_d455_joint" type="fixed">
-    <parent link="base_link" />
-    <child link="d455_link" />
-    <origin xyz="-0.115 0 0.525" rpy="0 0 3.14" />
-  </joint>
-  <joint name="d455_optical_joint" type="fixed">
-    <parent link="d455_link" />
-    <child link="d455_optical_link" />
-    <origin xyz="0 0 0" rpy="-1.5708 0 -1.5708" />
+    <origin xyz="0.08 0 0.8425" rpy="0 0 0" />
   </joint>
   <joint name="base_d456_joint" type="fixed">
     <parent link="base_link" />
     <child link="d456_link" />
-    <origin xyz="-0.04 0 0.525" rpy="0 0.523599 0" />
+    <origin xyz="0.0889 0 0.7975" rpy="0 0.523599 0" />
   </joint>
   <joint name="d456_optical_joint" type="fixed">
@@ -244,13 +161,4 @@
     <origin xyz="0 0 0" rpy="0 0 0" />
   </joint>
-  <gazebo reference="base_link">
-    <material>Gazebo/Grey</material>
-  </gazebo>
-  <gazebo reference="ebox_link">
-    <material>Gazebo/White</material>
-  </gazebo>
-  <gazebo reference="blade_link">
-    <material>Gazebo/Grey</material>
-  </gazebo>
   <gazebo reference="front_right_wheel_link">
     <material>Gazebo/DarkGrey</material>
@@ -312,42 +220,4 @@
       </contact>
     </surface>
-  </gazebo>
-  <gazebo reference="d455_link">
-    <sensor type="depth" name="d455">
-      <pose>0 0 0 0 0 0</pose>
-      <update_rate>30.0</update_rate>
-      <visualize>true</visualize>
-      <camera>
-        <horizontal_fov>1.540</horizontal_fov>
-        <image>
-          <width>640</width>
-          <height>360</height>
-          <format>R8G8B8</format>
-        </image>
-        <distortion>
-          <k1>-0.06792929080519726</k1>
-          <k2>0.08058277259698843</k2>
-          <k3>-0.04417756393089296</k3>
-          <p1>-0.001690544521662593</p1>
-          <p2>-0.0008235437909836152</p2>
-        </distortion>
-        <clip>
-          <near>0.05</near>
-          <far>10.0</far>
-        </clip>
-      </camera>
-      <plugin name="camera1_controller" filename="libgazebo_ros_camera.so">
-        <ros>
-          <remapping>/d455/image_raw:=/d455/color/image_raw</remapping>
-          <remapping>/d455/points:=/d455/color/points</remapping>
-          <remapping>/d455/camera_info:=/d455/color/camera_info</remapping>
-          <remapping>/d455/depth/image_raw:=/d455/depth/image_rect_raw</remapping>
-        </ros>
-        <frame_name>d455_optical_link</frame_name>
-        <publish_tf>false</publish_tf>
-        <publish_point_cloud>true</publish_point_cloud>
-      </plugin>
-    </sensor>
-    <material>Gazebo/Grey</material>
   </gazebo>
   <gazebo reference="d456_link">
@@ -450,5 +320,5 @@
       <robot_param>robot_description</robot_param>
       <robot_param_node>robot_state_publisher</robot_param_node>
-      <parameters>$(find lunabot_config)/params/gazebo_bulldozer_bot_params.yaml</parameters>
+      <parameters>$(find lunabot_config)/params/gazebo_trencher_bot_params.yaml</parameters>
     </plugin>
   </gazebo>
@@ -457,9 +327,4 @@
       <plugin>gazebo_ros2_control/GazeboSystem</plugin>
     </hardware>
-    <joint name="base_blade_joint">
-      <command_interface name="position" />
-      <state_interface name="position" />
-      <state_interface name="velocity" />
-    </joint>
     <joint name="base_front_right_wheel_joint">
       <command_interface name="velocity">
@@ -495,10 +360,3 @@
     </joint>
   </ros2_control>
-  <transmission name="transmission_base_blade_joint">
-    <plugin>transmission_interface/SimpleTransmission</plugin>
-    <actuator name="actuator_base_blade_joint" role="actuator_base_blade_joint" />
-    <joint name="base_blade_joint" role="base_blade_joint">
-      <mechanical_reduction>1.0</mechanical_reduction>
-    </joint>
-  </transmission>
 </robot>

Commit message: Fixed model path in rectangle_bot.xacro.

File: lunabot_simulation/urdf/robot/rectangle_bot.xacro (robot description, xacro)
@@ -22,5 +22,5 @@
     <visual>
       <geometry>
-        <mesh filename="file:///$(find lunabot_simulation)/models/rectangle_bot/rectangle_bot.stl" />
+        <mesh filename="file:///$(find lunabot_simulation)/models/rectangle_bot/rectangle_bot_body.stl" />
       </geometry>
       <origin xyz="0 0 0.1625" rpy="0 0 0" />
@@ -29,5 +29,5 @@
     <collision>
       <geometry>
-        <mesh filename="file:///$(find lunabot_simulation)/models/rectangle_bot/rectangle_bot.stl" />
+        <mesh filename="file:///$(find lunabot_simulation)/models/rectangle_bot/rectangle_bot_body.stl" />
       </geometry>
       <origin xyz="0 0 0.085" rpy="0 0 0" />

Commit message: Fixed sensor placement in rectangle_bot.xacro.

File: lunabot_simulation/urdf/robot/rectangle_bot.xacro (robot description, xacro)
@@ -193,5 +193,5 @@
     <parent link="base_link" />
     <child link="lidar_link" />
-    <origin xyz="-0.0925 0 0.405" rpy="0 0 0" />
+    <origin xyz="-0.075 0 0.575" rpy="0 0 0" />
   </joint>
   <joint name="base_blade_joint" type="revolute">
@@ -206,5 +206,5 @@
     <parent link="base_link" />
     <child link="d456_link" />
-    <origin xyz="-0.05 0 0.355" rpy="0 0.523599 0" />
+    <origin xyz="-0.04 0 0.525" rpy="0 0.523599 0" />
   </joint>
   <joint name="d456_optical_joint" type="fixed">
