Commit message: Added back rf2o_laser_odometry, added Foxglove Studio option for visualization, modified Nav2 and RTAB-Map parameters, fixed URDF descriptions, updated README.md.

File: lunabot_simulation/urdf/robot/simulation/realistic_rectangle_bot.xacro (robot description, xacro)
@@ -209,5 +209,5 @@
     <parent link="base_link" />
     <child link="lidar_link" />
-    <origin xyz="-0.075 0 0.575" rpy="0 0 0" />
+    <origin xyz="-0.0925 0 0.405" rpy="0 0 0" />
   </joint>
   <joint name="base_blade_joint" type="revolute">

File: lunabot_simulation/urdf/robot/simulation/rectangle_bot.xacro (robot description, xacro)
@@ -22,5 +22,5 @@
     <visual>
       <geometry>
-        <mesh filename="file:///$(find lunabot_simulation)/models/rectangle_bot/rectangle_bot.stl" />
+        <mesh filename="file:///$(find lunabot_simulation)/models/rectangle_bot/rectangle_bot_body.stl" />
       </geometry>
       <origin xyz="0 0 0.1625" rpy="0 0 0" />
@@ -29,5 +29,5 @@
     <collision>
       <geometry>
-        <mesh filename="file:///$(find lunabot_simulation)/models/rectangle_bot/rectangle_bot.stl" />
+        <mesh filename="file:///$(find lunabot_simulation)/models/rectangle_bot/rectangle_bot_body.stl" />
       </geometry>
       <origin xyz="0 0 0.085" rpy="0 0 0" />
@@ -209,5 +209,5 @@
     <parent link="base_link" />
     <child link="lidar_link" />
-    <origin xyz="-0.0925 0 0.405" rpy="0 0 0" />
+    <origin xyz="-0.075 0 0.575" rpy="0 0 0" />
   </joint>
   <joint name="base_blade_joint" type="revolute">
@@ -222,5 +222,5 @@
     <parent link="base_link" />
     <child link="d455_link" />
-    <origin xyz="-0.12 0 0.355" rpy="0 0 3.14" />
+    <origin xyz="-0.115 0 0.525" rpy="0 0 3.14" />
   </joint>
   <joint name="d455_optical_joint" type="fixed">
@@ -232,5 +232,5 @@
     <parent link="base_link" />
     <child link="d456_link" />
-    <origin xyz="-0.05 0 0.355" rpy="0 0.523599 0" />
+    <origin xyz="-0.04 0 0.525" rpy="0 0.523599 0" />
   </joint>
   <joint name="d456_optical_joint" type="fixed">

Commit message: Experimenting with odometry again, rf2o is fast but can drift especially with angles. ICP and rf2o together are likely the best combination alongside an IMU. Testing out UKF instead of EKF for odometry filtering. Cleaned up folder structure in lunabot_config. Removed lunar_surface mesh as collision in world files to allow robot to drive smoother. Added back the hard-coded alignment and driving code to construction zone, using Nav2 to navigate to the construction zone is too complex and unnecessary, leads to sometimes the robot facing the wrong direction. Using a straight path allows for smoother collection of the regolith. Updated README.md.

File: lunabot_simulation/urdf/robot/simulation/realistic_rectangle_bot.xacro (robot description, xacro)
@@ -209,5 +209,5 @@
     <parent link="base_link" />
     <child link="lidar_link" />
-    <origin xyz="-0.0925 0 0.405" rpy="0 0 0" />
+    <origin xyz="-0.075 0 0.575" rpy="0 0 0" />
   </joint>
   <joint name="base_blade_joint" type="revolute">
@@ -450,5 +450,5 @@
       <robot_param>robot_description</robot_param>
       <robot_param_node>robot_state_publisher</robot_param_node>
-      <parameters>$(find lunabot_config)/params/gazebo_bulldozer_bot_params.yaml</parameters>
+      <parameters>$(find lunabot_config)/params/gazebo/gazebo_bulldozer_bot_params.yaml</parameters>
     </plugin>
   </gazebo>

File: lunabot_simulation/urdf/robot/simulation/rectangle_bot.xacro (robot description, xacro)
@@ -450,5 +450,5 @@
       <robot_param>robot_description</robot_param>
       <robot_param_node>robot_state_publisher</robot_param_node>
-      <parameters>$(find lunabot_config)/params/gazebo_bulldozer_bot_params.yaml</parameters>
+      <parameters>$(find lunabot_config)/params/gazebo/gazebo_bulldozer_bot_params.yaml</parameters>
     </plugin>
   </gazebo>

File: lunabot_simulation/urdf/robot/simulation/square_bot.xacro (robot description, xacro)
@@ -419,5 +419,5 @@
       <robot_param>robot_description</robot_param>
       <robot_param_node>robot_state_publisher</robot_param_node>
-      <parameters>$(find lunabot_config)/params/gazebo_bulldozer_bot_params.yaml</parameters>
+      <parameters>$(find lunabot_config)/params/gazebo/gazebo_bulldozer_bot_params.yaml</parameters>
     </plugin>
   </gazebo>

File: lunabot_simulation/urdf/robot/simulation/trencher_bot.xacro (robot description, xacro)
@@ -384,5 +384,5 @@
       <robot_param>robot_description</robot_param>
       <robot_param_node>robot_state_publisher</robot_param_node>
-      <parameters>$(find lunabot_config)/params/gazebo_trencher_bot_params.yaml</parameters>
+      <parameters>$(find lunabot_config)/params/gazebo/gazebo_trencher_bot_params.yaml</parameters>
     </plugin>
   </gazebo>
