Commit message: Fixed major bugs with odometry, improved quality of navigation client, added new bulldozer model with functional blade joints, removed square and rectangle bot models, added models for two lidars, and modified rocks to be pushable in artemis worlds.

File: lunabot_simulation/urdf/robot/simulation/trencher_bot.xacro (robot description, xacro)
@@ -5,8 +5,8 @@
     <color rgba="0.61 0.61 0.61 1.0" />
   </material>
-  <material name="camera_grey">
+  <material name="camera_gray">
     <color rgba="0.81 0.81 0.81 1.0" />
   </material>
-  <material name="black">
+  <material name="lidar_black">
     <color rgba="0.22 0.22 0.22 1.0" />
   </material>
@@ -39,5 +39,5 @@
       </geometry>
       <origin xyz="0 0 0" rpy="0 0 -1.5708" />
-      <material name="black" />
+      <material name="lidar_black" />
     </visual>
     <collision>
@@ -54,5 +54,5 @@
       </geometry>
       <origin xyz="0 0 0" rpy="0 0 0" />
-      <material name="camera_grey" />
+      <material name="camera_gray" />
     </visual>
     <collision>
@@ -70,5 +70,5 @@
       </geometry>
       <origin xyz="0 0 0" rpy="0 0 0" />
-      <material name="camera_grey" />
+      <material name="camera_gray" />
     </visual>
     <collision>
@@ -356,5 +356,5 @@
       </plugin>
     </sensor>
-    <material>Gazebo/Black</material>
+    <material>Gazebo/lidar_black</material>
   </gazebo>
   <gazebo reference="imu_link">
