Commit message: Fixed bulldozer URDF and modified paths in launch files.

File: lunabot_simulation/urdf/robot/real/bulldozer_bot.xacro (robot description, xacro)
@@ -222,9 +222,4 @@
     <origin xyz="-0.125 0 0.5762" rpy="0 0 3.14" />
   </joint>
-  <joint name="d455_optical_joint" type="fixed">
-    <parent link="d455_link" />
-    <child link="d455_optical_link" />
-    <origin xyz="0 0 0" rpy="-1.5708 0 -1.5708" />
-  </joint>
   <joint name="base_d456_joint" type="fixed">
     <parent link="base_link" />
@@ -232,9 +227,4 @@
     <origin xyz="-0.0555 0 0.5762" rpy="0 0.523599 0" />
   </joint>
-  <joint name="d456_optical_joint" type="fixed">
-    <parent link="d456_link" />
-    <child link="d456_optical_link" />
-    <origin xyz="0 0 0" rpy="-1.5708 0 -1.5708" />
-  </joint>
   <joint name="base_s3_lidar_joint" type="fixed">
     <parent link="base_link" />

Commit message: Changing IMU filter to madgwick instead of complementary, rotated S3 lidar in URDF.

File: lunabot_simulation/urdf/robot/real/bulldozer_bot.xacro (robot description, xacro)
@@ -230,5 +230,5 @@
     <parent link="base_link" />
     <child link="s3_lidar_link" />
-    <origin xyz="-0.09025 0 0.6" rpy="0 0 0" />
+    <origin xyz="-0.09025 0 0.6" rpy="0 0 3.14" />
   </joint>
   <joint name="base_s2l_lidar_joint" type="fixed">
