Commit message: Odometry is now in 3D, working on tuning rgbd_odometry parameters. rgbd_odometry is less accurate position wise than icp_odometry but is capable of calculating more roll and pitch than IMU. Fixed more bugs in excavation_server, however, needs more PID tuning as it still oscillates.

File: lunabot_description/urdf/bulldozer_bot.urdf.xacro (robot description, xacro)
@@ -9,9 +9,11 @@
     <color rgba="0.22 0.22 0.22 1.0" />
   </material>
+  <!-- ================================= -->
+  <!--            BODY LINKS             -->
+  <!-- ================================= -->
   <link name="base_link">
     <visual>
       <geometry>
-        <mesh
-          filename="file:///$(find lunabot_description)/meshes/bulldozer_bot/bulldozer_bot_body.dae" />
+        <mesh filename="file:///$(find lunabot_description)/meshes/bulldozer_bot/bulldozer_bot_body.dae" />
       </geometry>
       <origin xyz="0 0 0.1625" rpy="0 0 1.5708" />
@@ -19,6 +21,5 @@
     <collision>
       <geometry>
-        <mesh
-          filename="file:///$(find lunabot_description)/meshes/bulldozer_bot/bulldozer_bot_body.stl" />
+        <mesh filename="file:///$(find lunabot_description)/meshes/bulldozer_bot/bulldozer_bot_body.stl" />
       </geometry>
       <origin xyz="0 0 0.1625" rpy="0 0 1.5708" />
@@ -33,6 +34,5 @@
     <visual>
       <geometry>
-        <mesh
-          filename="file:///$(find lunabot_description)/meshes/bulldozer_bot/bulldozer_bot_blade.dae" />
+        <mesh filename="file:///$(find lunabot_description)/meshes/bulldozer_bot/bulldozer_bot_blade.dae" />
       </geometry>
       <origin xyz="0 0 0" rpy="1.5708 0 1.5708" />
@@ -40,6 +40,5 @@
     <collision>
       <geometry>
-        <mesh
-          filename="file:///$(find lunabot_description)/meshes/bulldozer_bot/bulldozer_bot_blade.stl" />
+        <mesh filename="file:///$(find lunabot_description)/meshes/bulldozer_bot/bulldozer_bot_blade.stl" />
       </geometry>
       <origin xyz="0 0 0" rpy="1.5708 0 1.5708" />
@@ -54,6 +53,5 @@
     <visual>
       <geometry>
-        <mesh
-          filename="file:///$(find lunabot_description)/meshes/bulldozer_bot/bulldozer_bot_blade_arm.dae" />
+        <mesh filename="file:///$(find lunabot_description)/meshes/bulldozer_bot/bulldozer_bot_blade_arm.dae" />
       </geometry>
       <origin xyz="0.127 0 0" rpy="-1.5708 0 1.5708" />
@@ -61,6 +59,5 @@
     <collision>
       <geometry>
-        <mesh
-          filename="file:///$(find lunabot_description)/meshes/bulldozer_bot/bulldozer_bot_blade_arm.stl" />
+        <mesh filename="file:///$(find lunabot_description)/meshes/bulldozer_bot/bulldozer_bot_blade_arm.stl" />
       </geometry>
       <origin xyz="0.127 0 0" rpy="-1.5708 0 1.5708" />
@@ -72,4 +69,7 @@
     </inertial>
   </link>
+  <!-- ================================= -->
+  <!--           SENSOR LINKS            -->
+  <!-- ================================= -->
   <link name="d455_link">
     <visual>
@@ -135,4 +135,7 @@
   </link>
   <link name="imu_link"></link>
+  <!-- ================================= -->
+  <!--            WHEEL LINKS            -->
+  <!-- ================================= -->
   <link name="front_right_wheel_link">
     <inertial>
@@ -187,28 +190,7 @@
     </collision>
   </link>
-  <joint name="base_rear_right_wheel_joint" type="continuous">
-    <parent link="base_link" />
-    <child link="rear_right_wheel_link" />
-    <origin xyz="-0.235 -0.25 0.08" rpy="0 0 0" />
-    <axis xyz="0 1 0" />
-  </joint>
-  <joint name="base_rear_left_wheel_joint" type="continuous">
-    <parent link="base_link" />
-    <child link="rear_left_wheel_link" />
-    <origin xyz="-0.235 0.25 0.08" rpy="0 0 0" />
-    <axis xyz="0 1 0" />
-  </joint>
-  <joint name="base_front_right_wheel_joint" type="continuous">
-    <parent link="base_link" />
-    <child link="front_right_wheel_link" />
-    <origin xyz="0.215 -0.25 0.08" rpy="0 0 0" />
-    <axis xyz="0 1 0" />
-  </joint>
-  <joint name="base_front_left_wheel_joint" type="continuous">
-    <parent link="base_link" />
-    <child link="front_left_wheel_link" />
-    <origin xyz="0.215 0.25 0.08" rpy="0 0 0" />
-    <axis xyz="0 1 0" />
-  </joint>
+  <!-- ================================= -->
+  <!--            BODY JOINTS            -->
+  <!-- ================================= -->
   <joint name="base_blade_arm_joint" type="revolute">
     <parent link="base_link" />
@@ -227,4 +209,7 @@
     <dynamics damping="0.0" friction="0.0" />
   </joint>
+  <!-- ================================= -->
+  <!--           SENSOR JOINTS           -->
+  <!-- ================================= -->
   <joint name="base_d455_joint" type="fixed">
     <parent link="base_link" />
@@ -262,4 +247,34 @@
     <origin xyz="0 0 0" rpy="0 0 0" />
   </joint>
+  <!-- ================================= -->
+  <!--            WHEEL JOINTS           -->
+  <!-- ================================= -->
+  <joint name="base_rear_right_wheel_joint" type="continuous">
+    <parent link="base_link" />
+    <child link="rear_right_wheel_link" />
+    <origin xyz="-0.235 -0.25 0.08" rpy="0 0 0" />
+    <axis xyz="0 1 0" />
+  </joint>
+  <joint name="base_rear_left_wheel_joint" type="continuous">
+    <parent link="base_link" />
+    <child link="rear_left_wheel_link" />
+    <origin xyz="-0.235 0.25 0.08" rpy="0 0 0" />
+    <axis xyz="0 1 0" />
+  </joint>
+  <joint name="base_front_right_wheel_joint" type="continuous">
+    <parent link="base_link" />
+    <child link="front_right_wheel_link" />
+    <origin xyz="0.215 -0.25 0.08" rpy="0 0 0" />
+    <axis xyz="0 1 0" />
+  </joint>
+  <joint name="base_front_left_wheel_joint" type="continuous">
+    <parent link="base_link" />
+    <child link="front_left_wheel_link" />
+    <origin xyz="0.215 0.25 0.08" rpy="0 0 0" />
+    <axis xyz="0 1 0" />
+  </joint>
+  <!-- ================================= -->
+  <!--       GAZEBO CONFIGURATION        -->
+  <!-- ================================= -->
   <xacro:if value="$(arg use_sim)">
     <gazebo reference="front_right_wheel_link">

File: lunabot_description/urdf/trencher_bot.urdf.xacro (robot description, xacro)
@@ -15,4 +15,7 @@
     <color rgba="0.89 0.89 0.89 1.0" />
   </material>
+  <!-- ================================= -->
+  <!--            BODY LINKS             -->
+  <!-- ================================= -->
   <link name="base_link">
     <visual>
@@ -34,4 +37,7 @@
     </inertial>
   </link>
+  <!-- ================================= -->
+  <!--           SENSOR LINKS            -->
+  <!-- ================================= -->
   <link name="lidar_link">
     <visual>
@@ -82,4 +88,7 @@
   <link name="d456_optical_link"></link>
   <link name="imu_link"></link>
+  <!-- ================================= -->
+  <!--            WHEEL LINKS            -->
+  <!-- ================================= -->
   <link name="front_right_wheel_link">
     <inertial>
@@ -134,28 +143,10 @@
     </collision>
   </link>
-  <joint name="base_rear_right_wheel_joint" type="continuous">
-    <parent link="base_link" />
-    <child link="rear_right_wheel_link" />
-    <origin xyz="-0.305 -0.25 0.08" rpy="0 0 0" />
-    <axis xyz="0 1 0" />
-  </joint>
-  <joint name="base_rear_left_wheel_joint" type="continuous">
-    <parent link="base_link" />
-    <child link="rear_left_wheel_link" />
-    <origin xyz="-0.305 0.25 0.08" rpy="0 0 0" />
-    <axis xyz="0 1 0" />
-  </joint>
-  <joint name="base_front_right_wheel_joint" type="continuous">
-    <parent link="base_link" />
-    <child link="front_right_wheel_link" />
-    <origin xyz="0.1515 -0.25 0.08" rpy="0 0 0" />
-    <axis xyz="0 1 0" />
-  </joint>
-  <joint name="base_front_left_wheel_joint" type="continuous">
-    <parent link="base_link" />
-    <child link="front_left_wheel_link" />
-    <origin xyz="0.1515 0.25 0.08" rpy="0 0 0" />
-    <axis xyz="0 1 0" />
-  </joint>
+  <!-- ================================= -->
+  <!--            BODY JOINTS            -->
+  <!-- ================================= -->
+  <!-- ================================= -->
+  <!--           SENSOR JOINTS           -->
+  <!-- ================================= -->
   <joint name="base_lidar_joint" type="fixed">
     <parent link="base_link" />
@@ -188,4 +179,34 @@
     <origin xyz="0 0 0" rpy="0 0 0" />
   </joint>
+  <!-- ================================= -->
+  <!--            WHEEL JOINTS           -->
+  <!-- ================================= -->
+  <joint name="base_rear_right_wheel_joint" type="continuous">
+    <parent link="base_link" />
+    <child link="rear_right_wheel_link" />
+    <origin xyz="-0.305 -0.25 0.08" rpy="0 0 0" />
+    <axis xyz="0 1 0" />
+  </joint>
+  <joint name="base_rear_left_wheel_joint" type="continuous">
+    <parent link="base_link" />
+    <child link="rear_left_wheel_link" />
+    <origin xyz="-0.305 0.25 0.08" rpy="0 0 0" />
+    <axis xyz="0 1 0" />
+  </joint>
+  <joint name="base_front_right_wheel_joint" type="continuous">
+    <parent link="base_link" />
+    <child link="front_right_wheel_link" />
+    <origin xyz="0.1515 -0.25 0.08" rpy="0 0 0" />
+    <axis xyz="0 1 0" />
+  </joint>
+  <joint name="base_front_left_wheel_joint" type="continuous">
+    <parent link="base_link" />
+    <child link="front_left_wheel_link" />
+    <origin xyz="0.1515 0.25 0.08" rpy="0 0 0" />
+    <axis xyz="0 1 0" />
+  </joint>
+  <!-- ================================= -->
+  <!--       GAZEBO CONFIGURATION        -->
+  <!-- ================================= -->
   <xacro:if value="$(arg use_sim)">
     <gazebo reference="front_right_wheel_link">

Commit message: Modified bulldozer URDF, camera and lidar are now lined up.

File: lunabot_description/urdf/bulldozer_bot.urdf.xacro (robot description, xacro)
@@ -9,4 +9,12 @@
     <color rgba="0.22 0.22 0.22 1.0" />
   </material>
+  <xacro:if value="$(arg use_sim)">
+    <xacro:property name="camera_sim_link_offset" value="0.015" />
+    <xacro:property name="camera_sim_joint_offset" value="0" />
+  </xacro:if>
+  <xacro:unless value="$(arg use_sim)">
+    <xacro:property name="camera_sim_link_offset" value="0.15" />
+    <xacro:property name="camera_sim_joint_offset" value="0.15" />
+  </xacro:unless>
   <!-- ================================= -->
   <!--            BODY LINKS             -->
@@ -77,5 +85,5 @@
         <mesh filename="file:///$(find lunabot_description)/meshes/bulldozer_bot/bulldozer_bot_d455_camera.stl" />
       </geometry>
-      <origin xyz="0 0.015 0" rpy="0 0 0" />
+      <origin xyz="0 ${camera_sim_link_offset} 0" rpy="0 0 0" />
       <material name="camera_grey" />
     </visual>
@@ -84,5 +92,5 @@
         <mesh filename="file:///$(find lunabot_description)/meshes/bulldozer_bot/bulldozer_bot_d455_camera.stl" />
       </geometry>
-      <origin xyz="0 0.015 0" rpy="0 0 0" />
+      <origin xyz="0 ${camera_sim_link_offset} 0" rpy="0 0 0" />
     </collision>
   </link>
@@ -93,5 +101,5 @@
         <mesh filename="file:///$(find lunabot_description)/meshes/bulldozer_bot/bulldozer_bot_d456_camera.stl" />
       </geometry>
-      <origin xyz="0 -0.015 0" rpy="0 0 0" />
+      <origin xyz="0 -${camera_sim_link_offset} 0" rpy="0 0 0" />
       <material name="camera_grey" />
     </visual>
@@ -100,5 +108,5 @@
         <mesh filename="file:///$(find lunabot_description)/meshes/bulldozer_bot/bulldozer_bot_d456_camera.stl" />
       </geometry>
-      <origin xyz="0 -0.015 0" rpy="0 0 0" />
+      <origin xyz="0 -${camera_sim_link_offset} 0" rpy="0 0 0" />
     </collision>
   </link>
@@ -215,5 +223,5 @@
     <parent link="base_link" />
     <child link="d455_link" />
-    <origin xyz="-0.125 0 0.5762" rpy="0 0 3.14" />
+    <origin xyz="-0.125 -${camera_sim_joint_offset} 0.5762" rpy="0 0 3.14" />
   </joint>
   <joint name="d455_optical_joint" type="fixed">
@@ -225,5 +233,5 @@
     <parent link="base_link" />
     <child link="d456_link" />
-    <origin xyz="-0.0555 0 0.5762" rpy="0 0.523599 0" />
+    <origin xyz="-0.0555 ${camera_sim_joint_offset} 0.5762" rpy="0 0.523599 0" />
   </joint>
   <joint name="d456_optical_joint" type="fixed">

Commit message: Fixed D455 positioning in URDF.

File: lunabot_description/urdf/bulldozer_bot.urdf.xacro (robot description, xacro)
@@ -85,5 +85,5 @@
         <mesh filename="file:///$(find lunabot_description)/meshes/bulldozer_bot/bulldozer_bot_d455_camera.stl" />
       </geometry>
-      <origin xyz="0 ${camera_sim_link_offset} 0" rpy="0 0 0" />
+      <origin xyz="0 -${camera_sim_link_offset} 0" rpy="0 0 0" />
       <material name="camera_grey" />
     </visual>
@@ -92,5 +92,5 @@
         <mesh filename="file:///$(find lunabot_description)/meshes/bulldozer_bot/bulldozer_bot_d455_camera.stl" />
       </geometry>
-      <origin xyz="0 ${camera_sim_link_offset} 0" rpy="0 0 0" />
+      <origin xyz="0 -${camera_sim_link_offset} 0" rpy="0 0 0" />
     </collision>
   </link>

Commit message: Added OAK-D Pro and D435 to bulldozer model and modified real and sim launches to use these other cameras. Removed D455, using OAK-D instead since its IMU actually works. Using apriltag_ros instead of OpenCV for tag detection in localization_server.cpp.

File: lunabot_description/urdf/bulldozer_bot.urdf.xacro (robot description, xacro)
@@ -6,14 +6,18 @@
     <color rgba="0.81 0.81 0.81 1.0" />
   </material>
-  <material name="lidar_black">
+  <material name="black">
     <color rgba="0.22 0.22 0.22 1.0" />
   </material>
   <xacro:if value="$(arg use_sim)">
-    <xacro:property name="camera_sim_link_offset" value="0.015" />
-    <xacro:property name="camera_sim_joint_offset" value="0" />
+    <xacro:property name="d456_sim_link_offset" value="0.015" />
+    <xacro:property name="d456_sim_joint_offset" value="0" />
+    <xacro:property name="oak_d_sim_link_offset" value="0.015" />
+    <xacro:property name="oak_d_sim_joint_offset" value="0" />
+    <xacro:property name="d435_sim_link_offset" value="0.015" />
+    <xacro:property name="d435_sim_joint_offset" value="0" />
   </xacro:if>
   <xacro:unless value="$(arg use_sim)">
-    <xacro:property name="camera_sim_link_offset" value="0.15" />
-    <xacro:property name="camera_sim_joint_offset" value="0.15" />
+    <xacro:property name="d456_sim_link_offset" value="0.15" />
+    <xacro:property name="d456_sim_joint_offset" value="0.15" />
   </xacro:unless>
   <!-- ================================= -->
@@ -80,36 +84,52 @@
   <!--           SENSOR LINKS            -->
   <!-- ================================= -->
-  <link name="d455_link">
-    <visual>
-      <geometry>
-        <mesh filename="file:///$(find lunabot_description)/meshes/bulldozer_bot/bulldozer_bot_d455_camera.stl" />
-      </geometry>
-      <origin xyz="0 -${camera_sim_link_offset} 0" rpy="0 0 0" />
+  <link name="oak_d_link">
+    <visual>
+      <geometry>
+        <mesh filename="file:///$(find lunabot_description)/meshes/bulldozer_bot/bulldozer_bot_oak_d_camera.stl" />
+      </geometry>
+      <origin xyz="0 ${oak_d_sim_link_offset} 0" rpy="0 0 0" />
+      <material name="black" />
+    </visual>
+    <collision>
+      <geometry>
+        <mesh filename="file:///$(find lunabot_description)/meshes/bulldozer_bot/bulldozer_bot_oak_d_camera.stl" />
+      </geometry>
+      <origin xyz="0 ${oak_d_sim_link_offset} 0" rpy="0 0 0" />
+    </collision>
+  </link>
+  <link name="oak_d_optical_link"></link>
+  <link name="d456_link">
+    <visual>
+      <geometry>
+        <mesh filename="file:///$(find lunabot_description)/meshes/bulldozer_bot/bulldozer_bot_d456_camera.stl" />
+      </geometry>
+      <origin xyz="0 -${d456_sim_link_offset} 0" rpy="0 0 0" />
       <material name="camera_grey" />
     </visual>
     <collision>
       <geometry>
-        <mesh filename="file:///$(find lunabot_description)/meshes/bulldozer_bot/bulldozer_bot_d455_camera.stl" />
-      </geometry>
-      <origin xyz="0 -${camera_sim_link_offset} 0" rpy="0 0 0" />
-    </collision>
-  </link>
-  <link name="d455_optical_link"></link>
-  <link name="d456_link">
-    <visual>
-      <geometry>
         <mesh filename="file:///$(find lunabot_description)/meshes/bulldozer_bot/bulldozer_bot_d456_camera.stl" />
       </geometry>
-      <origin xyz="0 -${camera_sim_link_offset} 0" rpy="0 0 0" />
+      <origin xyz="0 -${d456_sim_link_offset} 0" rpy="0 0 0" />
+    </collision>
+  </link>
+  <link name="d456_optical_link"></link>
+    <link name="d435_link">
+    <visual>
+      <geometry>
+        <mesh filename="file:///$(find lunabot_description)/meshes/bulldozer_bot/bulldozer_bot_d435_camera.stl" />
+      </geometry>
+      <origin xyz="0 ${d435_sim_link_offset} 0" rpy="0 0 0" />
       <material name="camera_grey" />
     </visual>
     <collision>
       <geometry>
-        <mesh filename="file:///$(find lunabot_description)/meshes/bulldozer_bot/bulldozer_bot_d456_camera.stl" />
-      </geometry>
-      <origin xyz="0 -${camera_sim_link_offset} 0" rpy="0 0 0" />
-    </collision>
-  </link>
-  <link name="d456_optical_link"></link>
+        <mesh filename="file:///$(find lunabot_description)/meshes/bulldozer_bot/bulldozer_bot_d435_camera.stl" />
+      </geometry>
+      <origin xyz="0 ${d435_sim_link_offset} 0" rpy="0 0 0" />
+    </collision>
+  </link>
+  <link name="d435_optical_link"></link>
   <link name="s3_lidar_link">
     <visual>
@@ -118,5 +138,5 @@
       </geometry>
       <origin xyz="0 -0.0155 0" rpy="0 0 -1.5708" />
-      <material name="lidar_black" />
+      <material name="black" />
     </visual>
     <collision>
@@ -133,5 +153,5 @@
       </geometry>
       <origin xyz="0 -0.015 0" rpy="0 3.14 -1.5708" />
-      <material name="lidar_black" />
+      <material name="black" />
     </visual>
     <collision>
@@ -220,12 +240,12 @@
   <!--           SENSOR JOINTS           -->
   <!-- ================================= -->
-  <joint name="base_d455_joint" type="fixed">
-    <parent link="base_link" />
-    <child link="d455_link" />
-    <origin xyz="-0.125 -${camera_sim_joint_offset} 0.5762" rpy="0 0 3.14" />
-  </joint>
-  <joint name="d455_optical_joint" type="fixed">
-    <parent link="d455_link" />
-    <child link="d455_optical_link" />
+  <joint name="base_oak_d_joint" type="fixed">
+    <parent link="base_link" />
+    <child link="oak_d_link" />
+    <origin xyz="-0.128 0 0.5762" rpy="0 0 3.14" />
+  </joint>
+  <joint name="oak_d_optical_joint" type="fixed">
+    <parent link="oak_d_link" />
+    <child link="oak_d_optical_link" />
     <origin xyz="0 0 0" rpy="-1.5708 0 -1.5708" />
   </joint>
@@ -233,9 +253,19 @@
     <parent link="base_link" />
     <child link="d456_link" />
-    <origin xyz="-0.0555 ${camera_sim_joint_offset} 0.5762" rpy="0 0.523599 0" />
+    <origin xyz="-0.0555 ${d456_sim_joint_offset} 0.5762" rpy="0 0.523599 0" />
   </joint>
   <joint name="d456_optical_joint" type="fixed">
     <parent link="d456_link" />
     <child link="d456_optical_link" />
+    <origin xyz="0 0 0" rpy="-1.5708 0 -1.5708" />
+  </joint>
+    <joint name="base_d435_joint" type="fixed">
+    <parent link="base_link" />
+    <child link="d435_link" />
+    <origin xyz="-0.128 0 0.50" rpy="0 0.523599 3.14" />
+  </joint>
+  <joint name="d435_optical_joint" type="fixed">
+    <parent link="d435_link" />
+    <child link="d435_optical_link" />
     <origin xyz="0 0 0" rpy="-1.5708 0 -1.5708" />
   </joint>
@@ -346,11 +376,11 @@
       </surface>
     </gazebo>
-    <gazebo reference="d455_link">
-      <sensor type="depth" name="d455">
+    <gazebo reference="oak_d_link">
+      <sensor type="depth" name="oak_d">
         <pose>0 0 0 0 0 0</pose>
         <update_rate>60.0</update_rate>
         <visualize>true</visualize>
         <camera>
-          <horizontal_fov>1.540</horizontal_fov>
+          <horizontal_fov>1.434</horizontal_fov>
           <image>
             <width>640</width>
@@ -370,17 +400,17 @@
           </clip>
         </camera>
-        <plugin name="d455_controller" filename="libgazebo_ros_camera.so">
+        <plugin name="oak_d_controller" filename="libgazebo_ros_camera.so">
           <ros>
-            <remapping>/d455/image_raw:=/d455/color/image_raw</remapping>
-            <remapping>/d455/points:=/d455/color/points</remapping>
-            <remapping>/d455/camera_info:=/d455/color/camera_info</remapping>
-            <remapping>/d455/depth/image_raw:=/d455/depth/image_rect_raw</remapping>
+            <remapping>/oak_d/image_raw:=/oak_d/color/image_raw</remapping>
+            <remapping>/oak_d/points:=/oak_d/color/points</remapping>
+            <remapping>/oak_d/camera_info:=/oak_d/color/camera_info</remapping>
+            <remapping>/oak_d/depth/image_raw:=/oak_d/depth/image_rect_raw</remapping>
           </ros>
-          <frame_name>d455_optical_link</frame_name>
+          <frame_name>oak_d_optical_link</frame_name>
           <publish_tf>false</publish_tf>
           <publish_point_cloud>true</publish_point_cloud>
         </plugin>
       </sensor>
-      <material>Gazebo/Grey</material>
+      <material>Gazebo/Black</material>
     </gazebo>
     <gazebo reference="d456_link">
@@ -390,5 +420,5 @@
         <visualize>true</visualize>
         <camera>
-          <horizontal_fov>1.540</horizontal_fov>
+          <horizontal_fov>1.434</horizontal_fov>
           <image>
             <width>640</width>
@@ -416,4 +446,42 @@
           </ros>
           <frame_name>d456_optical_link</frame_name>
+          <publish_tf>false</publish_tf>
+          <publish_point_cloud>true</publish_point_cloud>
+        </plugin>
+      </sensor>
+      <material>Gazebo/Grey</material>
+    </gazebo>
+    <gazebo reference="d435_link">
+      <sensor type="depth" name="d435">
+        <pose>0 0 0 0 0 0</pose>
+        <update_rate>60.0</update_rate>
+        <visualize>true</visualize>
+        <camera>
+          <horizontal_fov>1.540</horizontal_fov>
+          <image>
+            <width>640</width>
+            <height>360</height>
+            <format>R8G8B8</format>
+          </image>
+          <distortion>
+            <k1>-0.06792929080519726</k1>
+            <k2>0.08058277259698843</k2>
+            <k3>-0.04417756393089296</k3>
+            <p1>-0.001690544521662593</p1>
+            <p2>-0.0008235437909836152</p2>
+          </distortion>
+          <clip>
+            <near>0.05</near>
+            <far>10.0</far>
+          </clip>
+        </camera>
+        <plugin name="d435_controller" filename="libgazebo_ros_camera.so">
+          <ros>
+            <remapping>/d435/image_raw:=/d435/color/image_raw</remapping>
+            <remapping>/d435/points:=/d435/color/points</remapping>
+            <remapping>/d435/camera_info:=/d435/color/camera_info</remapping>
+            <remapping>/d435/depth/image_raw:=/d435/depth/image_rect_raw</remapping>
+          </ros>
+          <frame_name>d435_optical_link</frame_name>
           <publish_tf>false</publish_tf>
           <publish_point_cloud>true</publish_point_cloud>
