Commit message: Fixed OAK-D Pro launching and added Depth AI dependencies script into install_dependencies.sh. Copied sim bot Nav2 params to real bot.

File: lunabot_description/urdf/bulldozer_bot.urdf.xacro (robot description, xacro)
@@ -20,4 +20,8 @@
     <xacro:property name="d456_sim_link_offset" value="0.15" />
     <xacro:property name="d456_sim_joint_offset" value="0.15" />
+    <xacro:property name="oak_d_sim_link_offset" value="0" />
+    <xacro:property name="oak_d_sim_joint_offset" value="0" />
+    <xacro:property name="d435_sim_link_offset" value="0" />
+    <xacro:property name="d435_sim_joint_offset" value="0" />
   </xacro:unless>
   <!-- ================================= -->

Commit message: Reformatting, added smoothing for driving and speed multipliers for both drive and blade movement. Added D455 camera to back to real_launch and URDF. Added new node to publish actuator position based off CAN messages sent from Teensy.

File: lunabot_description/urdf/bulldozer_bot.urdf.xacro (robot description, xacro)
@@ -10,18 +10,10 @@
   </material>
   <xacro:if value="$(arg use_sim)">
-    <xacro:property name="d456_sim_link_offset" value="0.015" />
-    <xacro:property name="d456_sim_joint_offset" value="0" />
-    <xacro:property name="oak_d_sim_link_offset" value="0.015" />
-    <xacro:property name="oak_d_sim_joint_offset" value="0" />
-    <xacro:property name="d435_sim_link_offset" value="0.015" />
-    <xacro:property name="d435_sim_joint_offset" value="0" />
+    <xacro:property name="camera_sim_link_offset" value="0.015" />
+    <xacro:property name="camera_sim_joint_offset" value="0" />
   </xacro:if>
   <xacro:unless value="$(arg use_sim)">
-    <xacro:property name="d456_sim_link_offset" value="0.15" />
-    <xacro:property name="d456_sim_joint_offset" value="0.15" />
-    <xacro:property name="oak_d_sim_link_offset" value="0" />
-    <xacro:property name="oak_d_sim_joint_offset" value="0" />
-    <xacro:property name="d435_sim_link_offset" value="0" />
-    <xacro:property name="d435_sim_joint_offset" value="0" />
+    <xacro:property name="camera_sim_link_offset" value="0.15" />
+    <xacro:property name="camera_sim_joint_offset" value="0.15" />
   </xacro:unless>
   <!-- ================================= -->
@@ -31,5 +23,6 @@
     <visual>
       <geometry>
-        <mesh filename="file:///$(find lunabot_description)/meshes/bulldozer_bot/bulldozer_bot_body.dae" />
+        <mesh
+          filename="file:///$(find lunabot_description)/meshes/bulldozer_bot/bulldozer_bot_body.dae" />
       </geometry>
       <origin xyz="0 0 0.1625" rpy="0 0 1.5708" />
@@ -37,5 +30,6 @@
     <collision>
       <geometry>
-        <mesh filename="file:///$(find lunabot_description)/meshes/bulldozer_bot/bulldozer_bot_body.stl" />
+        <mesh
+          filename="file:///$(find lunabot_description)/meshes/bulldozer_bot/bulldozer_bot_body.stl" />
       </geometry>
       <origin xyz="0 0 0.1625" rpy="0 0 1.5708" />
@@ -50,5 +44,6 @@
     <visual>
       <geometry>
-        <mesh filename="file:///$(find lunabot_description)/meshes/bulldozer_bot/bulldozer_bot_blade.dae" />
+        <mesh
+          filename="file:///$(find lunabot_description)/meshes/bulldozer_bot/bulldozer_bot_blade.dae" />
       </geometry>
       <origin xyz="0 0 0" rpy="1.5708 0 1.5708" />
@@ -56,5 +51,6 @@
     <collision>
       <geometry>
-        <mesh filename="file:///$(find lunabot_description)/meshes/bulldozer_bot/bulldozer_bot_blade.stl" />
+        <mesh
+          filename="file:///$(find lunabot_description)/meshes/bulldozer_bot/bulldozer_bot_blade.stl" />
       </geometry>
       <origin xyz="0 0 0" rpy="1.5708 0 1.5708" />
@@ -69,5 +65,6 @@
     <visual>
       <geometry>
-        <mesh filename="file:///$(find lunabot_description)/meshes/bulldozer_bot/bulldozer_bot_blade_arm.dae" />
+        <mesh
+          filename="file:///$(find lunabot_description)/meshes/bulldozer_bot/bulldozer_bot_blade_arm.dae" />
       </geometry>
       <origin xyz="0.127 0 0" rpy="-1.5708 0 1.5708" />
@@ -75,5 +72,6 @@
     <collision>
       <geometry>
-        <mesh filename="file:///$(find lunabot_description)/meshes/bulldozer_bot/bulldozer_bot_blade_arm.stl" />
+        <mesh
+          filename="file:///$(find lunabot_description)/meshes/bulldozer_bot/bulldozer_bot_blade_arm.stl" />
       </geometry>
       <origin xyz="0.127 0 0" rpy="-1.5708 0 1.5708" />
@@ -91,14 +89,16 @@
     <visual>
       <geometry>
-        <mesh filename="file:///$(find lunabot_description)/meshes/bulldozer_bot/bulldozer_bot_oak_d_camera.stl" />
-      </geometry>
-      <origin xyz="0 ${oak_d_sim_link_offset} 0" rpy="0 0 0" />
+        <mesh
+          filename="file:///$(find lunabot_description)/meshes/bulldozer_bot/bulldozer_bot_oak_d_camera.stl" />
+      </geometry>
+      <origin xyz="0 0 0" rpy="0 0 0" />
       <material name="black" />
     </visual>
     <collision>
       <geometry>
-        <mesh filename="file:///$(find lunabot_description)/meshes/bulldozer_bot/bulldozer_bot_oak_d_camera.stl" />
-      </geometry>
-      <origin xyz="0 ${oak_d_sim_link_offset} 0" rpy="0 0 0" />
+        <mesh
+          filename="file:///$(find lunabot_description)/meshes/bulldozer_bot/bulldozer_bot_oak_d_camera.stl" />
+      </geometry>
+      <origin xyz="0 0 0" rpy="0 0 0" />
     </collision>
   </link>
@@ -107,37 +107,42 @@
     <visual>
       <geometry>
-        <mesh filename="file:///$(find lunabot_description)/meshes/bulldozer_bot/bulldozer_bot_d456_camera.stl" />
-      </geometry>
-      <origin xyz="0 -${d456_sim_link_offset} 0" rpy="0 0 0" />
+        <mesh
+          filename="file:///$(find lunabot_description)/meshes/bulldozer_bot/bulldozer_bot_d456_camera.stl" />
+      </geometry>
+      <origin xyz="0 -${camera_sim_link_offset} 0" rpy="0 0 0" />
       <material name="camera_grey" />
     </visual>
     <collision>
       <geometry>
-        <mesh filename="file:///$(find lunabot_description)/meshes/bulldozer_bot/bulldozer_bot_d456_camera.stl" />
-      </geometry>
-      <origin xyz="0 -${d456_sim_link_offset} 0" rpy="0 0 0" />
+        <mesh
+          filename="file:///$(find lunabot_description)/meshes/bulldozer_bot/bulldozer_bot_d456_camera.stl" />
+      </geometry>
+      <origin xyz="0 -${camera_sim_link_offset} 0" rpy="0 0 0" />
     </collision>
   </link>
   <link name="d456_optical_link"></link>
-    <link name="d435_link">
-    <visual>
-      <geometry>
-        <mesh filename="file:///$(find lunabot_description)/meshes/bulldozer_bot/bulldozer_bot_d435_camera.stl" />
-      </geometry>
-      <origin xyz="0 ${d435_sim_link_offset} 0" rpy="0 0 0" />
+  <link name="d455_link">
+    <visual>
+      <geometry>
+        <mesh
+          filename="file:///$(find lunabot_description)/meshes/bulldozer_bot/bulldozer_bot_d455_camera.stl" />
+      </geometry>
+      <origin xyz="0 -${camera_sim_link_offset} 0" rpy="0 0 0" />
       <material name="camera_grey" />
     </visual>
     <collision>
       <geometry>
-        <mesh filename="file:///$(find lunabot_description)/meshes/bulldozer_bot/bulldozer_bot_d435_camera.stl" />
-      </geometry>
-      <origin xyz="0 ${d435_sim_link_offset} 0" rpy="0 0 0" />
-    </collision>
-  </link>
-  <link name="d435_optical_link"></link>
+        <mesh
+          filename="file:///$(find lunabot_description)/meshes/bulldozer_bot/bulldozer_bot_d455_camera.stl" />
+      </geometry>
+      <origin xyz="0 -${camera_sim_link_offset} 0" rpy="0 0 0" />
+    </collision>
+  </link>
+  <link name="d455_optical_link"></link>
   <link name="s3_lidar_link">
     <visual>
       <geometry>
-        <mesh filename="file:///$(find lunabot_description)/meshes/bulldozer_bot/bulldozer_bot_s3_lidar.stl" />
+        <mesh
+          filename="file:///$(find lunabot_description)/meshes/bulldozer_bot/bulldozer_bot_s3_lidar.stl" />
       </geometry>
       <origin xyz="0 -0.0155 0" rpy="0 0 -1.5708" />
@@ -146,5 +151,6 @@
     <collision>
       <geometry>
-        <mesh filename="file:///$(find lunabot_description)/meshes/bulldozer_bot/bulldozer_bot_s3_lidar.stl" />
+        <mesh
+          filename="file:///$(find lunabot_description)/meshes/bulldozer_bot/bulldozer_bot_s3_lidar.stl" />
       </geometry>
       <origin xyz="0 -0.0155 0" rpy="0 0 -1.5708" />
@@ -154,5 +160,6 @@
     <visual>
       <geometry>
-        <mesh filename="file:///$(find lunabot_description)/meshes/bulldozer_bot/bulldozer_bot_s2l_lidar.stl" />
+        <mesh
+          filename="file:///$(find lunabot_description)/meshes/bulldozer_bot/bulldozer_bot_s2l_lidar.stl" />
       </geometry>
       <origin xyz="0 -0.015 0" rpy="0 3.14 -1.5708" />
@@ -161,5 +168,6 @@
     <collision>
       <geometry>
-        <mesh filename="file:///$(find lunabot_description)/meshes/bulldozer_bot/bulldozer_bot_s2l_lidar.stl" />
+        <mesh
+          filename="file:///$(find lunabot_description)/meshes/bulldozer_bot/bulldozer_bot_s2l_lidar.stl" />
       </geometry>
       <origin xyz="0 -0.015 0" rpy="0 0 -1.5708" />
@@ -247,5 +255,5 @@
     <parent link="base_link" />
     <child link="oak_d_link" />
-    <origin xyz="-0.128 0 0.5762" rpy="0 0 3.14" />
+    <origin xyz="-0.128 0 0.50" rpy="0 0 3.14" />
   </joint>
   <joint name="oak_d_optical_joint" type="fixed">
@@ -254,22 +262,22 @@
     <origin xyz="0 0 0" rpy="-1.5708 0 -1.5708" />
   </joint>
+  <joint name="base_d455_joint" type="fixed">
+    <parent link="base_link" />
+    <child link="d455_link" />
+    <origin xyz="-0.128 -${camera_sim_joint_offset} 0.5762" rpy="0 0.785398 3.14" />
+  </joint>
+  <joint name="d455_optical_joint" type="fixed">
+    <parent link="d455_link" />
+    <child link="d455_optical_link" />
+    <origin xyz="0 0 0" rpy="-1.5708 0 -1.5708" />
+  </joint>
   <joint name="base_d456_joint" type="fixed">
     <parent link="base_link" />
     <child link="d456_link" />
-    <origin xyz="-0.0555 ${d456_sim_joint_offset} 0.5762" rpy="0 0.523599 0" />
+    <origin xyz="-0.0555 ${camera_sim_joint_offset} 0.5762" rpy="0 0.523599 0" />
   </joint>
   <joint name="d456_optical_joint" type="fixed">
     <parent link="d456_link" />
     <child link="d456_optical_link" />
-    <origin xyz="0 0 0" rpy="-1.5708 0 -1.5708" />
-  </joint>
-    <joint name="base_d435_joint" type="fixed">
-    <parent link="base_link" />
-    <child link="d435_link" />
-    <origin xyz="-0.128 0 0.50" rpy="0 0.523599 3.14" />
-  </joint>
-  <joint name="d435_optical_joint" type="fixed">
-    <parent link="d435_link" />
-    <child link="d435_optical_link" />
     <origin xyz="0 0 0" rpy="-1.5708 0 -1.5708" />
   </joint>
@@ -456,6 +464,6 @@
       <material>Gazebo/Grey</material>
     </gazebo>
-    <gazebo reference="d435_link">
-      <sensor type="depth" name="d435">
+    <gazebo reference="d455_link">
+      <sensor type="depth" name="d455">
         <pose>0 0 0 0 0 0</pose>
         <update_rate>60.0</update_rate>
@@ -480,12 +488,12 @@
           </clip>
         </camera>
-        <plugin name="d435_controller" filename="libgazebo_ros_camera.so">
+        <plugin name="d455_controller" filename="libgazebo_ros_camera.so">
           <ros>
-            <remapping>/d435/image_raw:=/d435/color/image_raw</remapping>
-            <remapping>/d435/points:=/d435/color/points</remapping>
-            <remapping>/d435/camera_info:=/d435/color/camera_info</remapping>
-            <remapping>/d435/depth/image_raw:=/d435/depth/image_rect_raw</remapping>
+            <remapping>/d455/image_raw:=/d455/color/image_raw</remapping>
+            <remapping>/d455/points:=/d455/color/points</remapping>
+            <remapping>/d455/camera_info:=/d455/color/camera_info</remapping>
+            <remapping>/d455/depth/image_raw:=/d455/depth/image_rect_raw</remapping>
           </ros>
-          <frame_name>d435_optical_link</frame_name>
+          <frame_name>d455_optical_link</frame_name>
           <publish_tf>false</publish_tf>
           <publish_point_cloud>true</publish_point_cloud>

Commit message: Added heartbeat back in, modified real_launch for new camera positions.

File: lunabot_description/urdf/bulldozer_bot.urdf.xacro (robot description, xacro)
@@ -255,5 +255,5 @@
     <parent link="base_link" />
     <child link="oak_d_link" />
-    <origin xyz="-0.128 0 0.50" rpy="0 0 3.14" />
+    <origin xyz="-0.128 0 0.5762" rpy="0 0.785398 3.14" />
   </joint>
   <joint name="oak_d_optical_joint" type="fixed">
@@ -265,5 +265,5 @@
     <parent link="base_link" />
     <child link="d455_link" />
-    <origin xyz="-0.128 -${camera_sim_joint_offset} 0.5762" rpy="0 0.785398 3.14" />
+    <origin xyz="-0.128 -${camera_sim_joint_offset} 0.5" rpy="0 0 3.14" />
   </joint>
   <joint name="d455_optical_joint" type="fixed">

Commit message: Testing autonomy, IMU on Teensy is fully functional and mapping has improved on rough terrain. Fixed bugs with AprilTag localization. Added node to read data from Teensy and publish encoder position and IMU data.

File: lunabot_description/urdf/bulldozer_bot.urdf.xacro (robot description, xacro)
@@ -295,5 +295,5 @@
     <parent link="base_link" />
     <child link="imu_link" />
-    <origin xyz="0 0 0" rpy="0 0 0" />
+    <origin xyz="0 0 0" rpy="3.14159 0 -1.57" />
   </joint>
   <!-- ================================= -->

Commit message: Modified coordinates for UCF arena.

File: lunabot_description/urdf/bulldozer_bot.urdf.xacro (robot description, xacro)
@@ -295,5 +295,5 @@
     <parent link="base_link" />
     <child link="imu_link" />
-    <origin xyz="0 0 0" rpy="0 0 0" />
+    <origin xyz="0 0 0" rpy="3.14159 0 -1.57" />
   </joint>
   <!-- ================================= -->
@@ -581,5 +581,5 @@
           <ros>
             <namespace></namespace>
-            <remapping>~/out:=/d456/imu/data</remapping>
+            <remapping>~/out:=/teensy/imu/data</remapping>
           </ros>
           <bodyName>base_link</bodyName>

Commit message: Removed dual camera mapping setup in preparation for adding 3D lidar, much faster to build now without needing to build RTAB-Map from source. Added UCF arena. Added some 3D lidar submodules.

File: lunabot_description/urdf/bulldozer_bot.urdf.xacro (robot description, xacro)
@@ -122,22 +122,4 @@
   </link>
   <link name="d456_optical_link"></link>
-  <link name="d455_link">
-    <visual>
-      <geometry>
-        <mesh
-          filename="file:///$(find lunabot_description)/meshes/bulldozer_bot/bulldozer_bot_d455_camera.stl" />
-      </geometry>
-      <origin xyz="0 -${camera_sim_link_offset} 0" rpy="0 0 0" />
-      <material name="camera_grey" />
-    </visual>
-    <collision>
-      <geometry>
-        <mesh
-          filename="file:///$(find lunabot_description)/meshes/bulldozer_bot/bulldozer_bot_d455_camera.stl" />
-      </geometry>
-      <origin xyz="0 -${camera_sim_link_offset} 0" rpy="0 0 0" />
-    </collision>
-  </link>
-  <link name="d455_optical_link"></link>
   <link name="s3_lidar_link">
     <visual>
@@ -155,21 +137,4 @@
       </geometry>
       <origin xyz="0 -0.0155 0" rpy="0 0 -1.5708" />
-    </collision>
-  </link>
-  <link name="s2l_lidar_link">
-    <visual>
-      <geometry>
-        <mesh
-          filename="file:///$(find lunabot_description)/meshes/bulldozer_bot/bulldozer_bot_s2l_lidar.stl" />
-      </geometry>
-      <origin xyz="0 -0.015 0" rpy="0 3.14 -1.5708" />
-      <material name="black" />
-    </visual>
-    <collision>
-      <geometry>
-        <mesh
-          filename="file:///$(find lunabot_description)/meshes/bulldozer_bot/bulldozer_bot_s2l_lidar.stl" />
-      </geometry>
-      <origin xyz="0 -0.015 0" rpy="0 0 -1.5708" />
     </collision>
   </link>
@@ -262,18 +227,8 @@
     <origin xyz="0 0 0" rpy="-1.5708 0 -1.5708" />
   </joint>
-  <joint name="base_d455_joint" type="fixed">
-    <parent link="base_link" />
-    <child link="d455_link" />
+  <joint name="base_d456_joint" type="fixed">
+    <parent link="base_link" />
+    <child link="d456_link" />
     <origin xyz="-0.128 -${camera_sim_joint_offset} 0.5" rpy="0 0 3.14" />
-  </joint>
-  <joint name="d455_optical_joint" type="fixed">
-    <parent link="d455_link" />
-    <child link="d455_optical_link" />
-    <origin xyz="0 0 0" rpy="-1.5708 0 -1.5708" />
-  </joint>
-  <joint name="base_d456_joint" type="fixed">
-    <parent link="base_link" />
-    <child link="d456_link" />
-    <origin xyz="-0.0555 ${camera_sim_joint_offset} 0.5762" rpy="0 0.523599 0" />
   </joint>
   <joint name="d456_optical_joint" type="fixed">
@@ -287,13 +242,8 @@
     <origin xyz="-0.09025 0 0.6" rpy="0 0 0" />
   </joint>
-  <joint name="base_s2l_lidar_joint" type="fixed">
-    <parent link="base_link" />
-    <child link="s2l_lidar_link" />
-    <origin xyz="0.26 0 0.175" rpy="0 0 0" />
-  </joint>
   <joint name="imu_joint" type="fixed">
     <parent link="base_link" />
     <child link="imu_link" />
-    <origin xyz="0 0 0" rpy="3.14159 0 -1.57" />
+    <origin xyz="0 0 0" rpy="0 0 0" />
   </joint>
   <!-- ================================= -->
@@ -432,5 +382,5 @@
         <visualize>true</visualize>
         <camera>
-          <horizontal_fov>1.434</horizontal_fov>
+          <horizontal_fov>1.540</horizontal_fov>
           <image>
             <width>640</width>
@@ -458,42 +408,4 @@
           </ros>
           <frame_name>d456_optical_link</frame_name>
-          <publish_tf>false</publish_tf>
-          <publish_point_cloud>true</publish_point_cloud>
-        </plugin>
-      </sensor>
-      <material>Gazebo/Grey</material>
-    </gazebo>
-    <gazebo reference="d455_link">
-      <sensor type="depth" name="d455">
-        <pose>0 0 0 0 0 0</pose>
-        <update_rate>60.0</update_rate>
-        <visualize>true</visualize>
-        <camera>
-          <horizontal_fov>1.540</horizontal_fov>
-          <image>
-            <width>640</width>
-            <height>360</height>
-            <format>R8G8B8</format>
-          </image>
-          <distortion>
-            <k1>-0.06792929080519726</k1>
-            <k2>0.08058277259698843</k2>
-            <k3>-0.04417756393089296</k3>
-            <p1>-0.001690544521662593</p1>
-            <p2>-0.0008235437909836152</p2>
-          </distortion>
-          <clip>
-            <near>0.05</near>
-            <far>10.0</far>
-          </clip>
-        </camera>
-        <plugin name="d455_controller" filename="libgazebo_ros_camera.so">
-          <ros>
-            <remapping>/d455/image_raw:=/d455/color/image_raw</remapping>
-            <remapping>/d455/points:=/d455/color/points</remapping>
-            <remapping>/d455/camera_info:=/d455/color/camera_info</remapping>
-            <remapping>/d455/depth/image_raw:=/d455/depth/image_rect_raw</remapping>
-          </ros>
-          <frame_name>d455_optical_link</frame_name>
           <publish_tf>false</publish_tf>
           <publish_point_cloud>true</publish_point_cloud>
@@ -537,39 +449,4 @@
       <material>Gazebo/Black</material>
     </gazebo>
-    <gazebo reference="s2l_lidar_link">
-      <sensor type="ray" name="s2l_lidar_link">
-        <pose>0 0 0 0 0 0</pose>
-        <visualize>false</visualize>
-        <update_rate>20.0</update_rate>
-        <ray>
-          <scan>
-            <horizontal>
-              <samples>1080</samples>
-              <resolution>0.5</resolution>
-              <min_angle>-3.14</min_angle>
-              <max_angle>3.14</max_angle>
-            </horizontal>
-          </scan>
-          <range>
-            <min>0.1</min>
-            <max>10.0</max>
-          </range>
-          <noise>
-            <type>gaussian</type>
-            <mean>0.0</mean>
-            <stddev>0.01</stddev>
-          </noise>
-        </ray>
-        <plugin name="s2l_lidar_controller" filename="libgazebo_ros_ray_sensor.so">
-          <frame_name>s2l_lidar_link</frame_name>
-          <ros>
-            <remapping>~/out:=/scan2_raw</remapping>
-          </ros>
-          <output_type>sensor_msgs/LaserScan</output_type>
-          <publish_tf>false</publish_tf>
-        </plugin>
-      </sensor>
-      <material>Gazebo/Black</material>
-    </gazebo>
     <gazebo reference="imu_link">
       <gravity>false</gravity>
@@ -581,5 +458,5 @@
           <ros>
             <namespace></namespace>
-            <remapping>~/out:=/teensy/imu/data</remapping>
+            <remapping>~/out:=/imu/data</remapping>
           </ros>
           <bodyName>base_link</bodyName>
