Commit message: Removed OAK-D link from URDF.

File: lunabot_description/urdf/bulldozer_bot.urdf.xacro (robot description, xacro)
@@ -86,22 +86,4 @@
   <!--           SENSOR LINKS            -->
   <!-- ================================= -->
-  <link name="oak_d_link">
-    <visual>
-      <geometry>
-        <mesh
-          filename="file:///$(find lunabot_description)/meshes/bulldozer_bot/bulldozer_bot_oak_d_camera.stl" />
-      </geometry>
-      <origin xyz="0 0 0" rpy="0 0 0" />
-      <material name="black" />
-    </visual>
-    <collision>
-      <geometry>
-        <mesh
-          filename="file:///$(find lunabot_description)/meshes/bulldozer_bot/bulldozer_bot_oak_d_camera.stl" />
-      </geometry>
-      <origin xyz="0 0 0" rpy="0 0 0" />
-    </collision>
-  </link>
-  <link name="oak_d_optical_link"></link>
   <link name="d456_link">
     <visual>
@@ -217,14 +199,4 @@
   <!--           SENSOR JOINTS           -->
   <!-- ================================= -->
-  <joint name="base_oak_d_joint" type="fixed">
-    <parent link="base_link" />
-    <child link="oak_d_link" />
-    <origin xyz="-0.128 0 0.5762" rpy="0 0.785398 3.14" />
-  </joint>
-  <joint name="oak_d_optical_joint" type="fixed">
-    <parent link="oak_d_link" />
-    <child link="oak_d_optical_link" />
-    <origin xyz="0 0 0" rpy="-1.5708 0 -1.5708" />
-  </joint>
   <joint name="base_d456_joint" type="fixed">
     <parent link="base_link" />
@@ -337,42 +309,4 @@
         </contact>
       </surface>
-    </gazebo>
-    <gazebo reference="oak_d_link">
-      <sensor type="depth" name="oak_d">
-        <pose>0 0 0 0 0 0</pose>
-        <update_rate>60.0</update_rate>
-        <visualize>true</visualize>
-        <camera>
-          <horizontal_fov>1.434</horizontal_fov>
-          <image>
-            <width>640</width>
-            <height>360</height>
-            <format>R8G8B8</format>
-          </image>
-          <distortion>
-            <k1>-0.06792929080519726</k1>
-            <k2>0.08058277259698843</k2>
-            <k3>-0.04417756393089296</k3>
-            <p1>-0.001690544521662593</p1>
-            <p2>-0.0008235437909836152</p2>
-          </distortion>
-          <clip>
-            <near>0.05</near>
-            <far>10.0</far>
-          </clip>
-        </camera>
-        <plugin name="oak_d_controller" filename="libgazebo_ros_camera.so">
-          <ros>
-            <remapping>/oak_d/image_raw:=/oak_d/color/image_raw</remapping>
-            <remapping>/oak_d/points:=/oak_d/color/points</remapping>
-            <remapping>/oak_d/camera_info:=/oak_d/color/camera_info</remapping>
-            <remapping>/oak_d/depth/image_raw:=/oak_d/depth/image_rect_raw</remapping>
-          </ros>
-          <frame_name>oak_d_optical_link</frame_name>
-          <publish_tf>false</publish_tf>
-          <publish_point_cloud>true</publish_point_cloud>
-        </plugin>
-      </sensor>
-      <material>Gazebo/Black</material>
     </gazebo>
     <gazebo reference="d456_link">

Commit message: Added Livox Mid-360 simulation support and added test bot model.

File: lunabot_description/urdf/bulldozer_bot.urdf.xacro (robot description, xacro)
@@ -104,22 +104,20 @@
   </link>
   <link name="d456_optical_link"></link>
-  <link name="s3_lidar_link">
+  <link name="mid360_lidar_link">
     <visual>
       <geometry>
         <mesh
-          filename="file:///$(find lunabot_description)/meshes/bulldozer_bot/bulldozer_bot_s3_lidar.stl" />
-      </geometry>
-      <origin xyz="0 -0.0155 0" rpy="0 0 -1.5708" />
-      <material name="black" />
+          filename="file:///$(find lunabot_description)/meshes/bulldozer_bot/bulldozer_bot_mid360_lidar.stl" />
+      </geometry>
+      <material name="camera_grey" />
     </visual>
     <collision>
       <geometry>
         <mesh
-          filename="file:///$(find lunabot_description)/meshes/bulldozer_bot/bulldozer_bot_s3_lidar.stl" />
-      </geometry>
-      <origin xyz="0 -0.0155 0" rpy="0 0 -1.5708" />
-    </collision>
-  </link>
-  <link name="imu_link"></link>
+          filename="file:///$(find lunabot_description)/meshes/bulldozer_bot/bulldozer_bot_mid360_lidar.stl" />
+      </geometry>
+    </collision>
+  </link>
+  <link name="mid360_imu_link"></link>
   <!-- ================================= -->
   <!--            WHEEL LINKS            -->
@@ -209,12 +207,12 @@
     <origin xyz="0 0 0" rpy="-1.5708 0 -1.5708" />
   </joint>
-  <joint name="base_s3_lidar_joint" type="fixed">
-    <parent link="base_link" />
-    <child link="s3_lidar_link" />
+  <joint name="base_mid360_joint" type="fixed">
+    <parent link="base_link" />
+    <child link="mid360_lidar_link" />
     <origin xyz="-0.09025 0 0.6" rpy="0 0 0" />
   </joint>
-  <joint name="imu_joint" type="fixed">
-    <parent link="base_link" />
-    <child link="imu_link" />
+  <joint name="mid360_imu_joint" type="fixed">
+    <parent link="mid360_lidar_link" />
+    <child link="mid360_imu_link" />
     <origin xyz="0 0 0" rpy="0 0 0" />
   </joint>
@@ -348,40 +346,46 @@
       <material>Gazebo/Grey</material>
     </gazebo>
-    <gazebo reference="s3_lidar_link">
-      <sensor type="ray" name="s3_lidar_link">
+    <gazebo reference="mid360_lidar_link">
+      <sensor type="ray" name="mid360_lidar_link">
+        <always_on>true</always_on>
         <pose>0 0 0 0 0 0</pose>
-        <visualize>false</visualize>
-        <update_rate>20.0</update_rate>
-        <ray>
-          <scan>
-            <horizontal>
-              <samples>1080</samples>
-              <resolution>0.5</resolution>
-              <min_angle>-3.14</min_angle>
-              <max_angle>3.14</max_angle>
-            </horizontal>
-          </scan>
-          <range>
-            <min>0.1</min>
-            <max>10.0</max>
-          </range>
-          <noise>
-            <type>gaussian</type>
-            <mean>0.0</mean>
-            <stddev>0.01</stddev>
-          </noise>
-        </ray>
-        <plugin name="s3_lidar_controller" filename="libgazebo_ros_ray_sensor.so">
-          <frame_name>s3_lidar_link</frame_name>
-          <ros>
-            <remapping>~/out:=/scan_raw</remapping>
-          </ros>
-          <output_type>sensor_msgs/LaserScan</output_type>
-          <publish_tf>false</publish_tf>
+        <visualize>true</visualize>
+        <update_rate>10</update_rate>
+        <plugin name="mid360_plugin" filename="libros2_livox.so">
+          <ray>
+            <scan>
+              <horizontal>
+                <samples>100</samples>
+                <resolution>1</resolution>
+                <min_angle>0</min_angle>
+                <max_angle>6.2831852</max_angle>
+              </horizontal>
+              <vertical>
+                <samples>360</samples>
+                <resolution>1</resolution>
+                <min_angle>-0.126</min_angle>
+                <max_angle>0.964</max_angle>
+              </vertical>
+            </scan>
+            <range>
+              <min>0.1</min>
+              <max>200.0</max>
+              <resolution>0.002</resolution>
+            </range>
+            <noise>
+              <type>gaussian</type>
+              <mean>0.0</mean>
+              <stddev>0.01</stddev>
+            </noise>
+          </ray>
+          <visualize>false</visualize>
+          <samples>30000</samples>
+          <downsample>1</downsample>
+          <csv_file_name>$(find ros2_livox_simulation)/scan_mode/mid360.csv</csv_file_name>
+          <topic>livox</topic>
         </plugin>
       </sensor>
-      <material>Gazebo/Black</material>
-    </gazebo>
-    <gazebo reference="imu_link">
+    </gazebo>
+    <gazebo reference="mid360_imu_link">
       <gravity>false</gravity>
       <sensor name="imu_sensor" type="imu">
@@ -392,5 +396,5 @@
           <ros>
             <namespace></namespace>
-            <remapping>~/out:=/imu/data</remapping>
+            <remapping>~/out:=/livox/imu</remapping>
           </ros>
           <bodyName>base_link</bodyName>
@@ -398,5 +402,5 @@
           <xyzOffset>0 0 0</xyzOffset>
           <rpyOffset>0 0 0</rpyOffset>
-          <frameName>imu_link</frameName>
+          <frameName>mid360_imu_link</frameName>
           <publish_tf>false</publish_tf>
           <initialOrientationAsReference>false</initialOrientationAsReference>
