Commit message: Working upside down lidar, still tuning rtabmap

File: lunabot_description/urdf/v2.urdf.xacro (robot description, xacro)
@@ -198,10 +198,10 @@
     <parent link="base_link" />
     <child link="mid360_lidar_link" />
-    <origin xyz="-0.27 0 0.548" rpy="0 0 0" />
+    <origin xyz="-0.27 0 0.548" rpy="3.14159 0 0" />
   </joint>
   <joint name="mid360_imu_joint" type="fixed">
     <parent link="base_link" />
     <child link="mid360_imu_link" />
-    <origin xyz="-0.27 0 0.548" rpy="0 0 0" />
+    <origin xyz="-0.27 0 0.548" rpy="3.14159 0 0" />
   </joint>
   <!-- ================================= -->
