Commit message: Changed lidar frame name

File: lunabot_description/urdf/v1_bot.urdf.xacro (robot description, xacro)
@@ -80,5 +80,5 @@
   </link>
   <link name="camera_back_optical_link"></link>
-  <link name="mid360_lidar_link">
+  <link name="livox_frame">
     <visual>
       <geometry>
@@ -176,5 +176,5 @@
   <joint name="base_mid360_joint" type="fixed">
     <parent link="base_link" />
-    <child link="mid360_lidar_link" />
+    <child link="livox_frame" />
     <origin xyz="-0.128 0 0.46" rpy="0 0 0" />
   </joint>
@@ -351,6 +351,6 @@
       <material>Gazebo/Grey</material>
     </gazebo>
-    <gazebo reference="mid360_lidar_link">
-      <sensor type="ray" name="mid360_lidar_link">
+    <gazebo reference="livox_frame">
+      <sensor type="ray" name="mid360_lidar_sensor">
         <always_on>true</always_on>
         <pose>0 0 0 0 0 0</pose>

File: lunabot_description/urdf/v2_bot.urdf.xacro (robot description, xacro)
@@ -130,5 +130,5 @@
   </link>
   <link name="camera_fisheye_optical_link"></link>
-  <link name="mid360_lidar_link">
+  <link name="livox_frame">
     <visual>
       <geometry>
@@ -244,5 +244,5 @@
   <joint name="base_mid360_joint" type="fixed">
     <parent link="base_link" />
-    <child link="mid360_lidar_link" />
+    <child link="livox_frame" />
     <origin xyz="-0.27 0 0.548" rpy="3.14159 0 0" />
   </joint>
@@ -468,6 +468,6 @@
       <material>Gazebo/Grey</material>
     </gazebo>
-    <gazebo reference="mid360_lidar_link">
-      <sensor type="ray" name="mid360_lidar_link">
+    <gazebo reference="livox_frame">
+      <sensor type="ray" name="mid360_lidar_sensor">
         <always_on>true</always_on>
         <pose>0 0 0 0 0 0</pose>

Commit message: Fixed lidar orientation

File: lunabot_description/urdf/v1_bot.urdf.xacro (robot description, xacro)
@@ -177,5 +177,5 @@
     <parent link="base_link" />
     <child link="livox_frame" />
-    <origin xyz="-0.128 0 0.46" rpy="0 0 0" />
+    <origin xyz="-0.128 0 0.46" rpy="3.14159 0 -1.5708" />
   </joint>
   <joint name="mid360_imu_joint" type="fixed">

File: lunabot_description/urdf/v2_bot.urdf.xacro (robot description, xacro)
@@ -245,5 +245,5 @@
     <parent link="base_link" />
     <child link="livox_frame" />
-    <origin xyz="-0.27 0 0.548" rpy="3.14159 0 0" />
+    <origin xyz="-0.27 0 0.548" rpy="3.14159 0 -1.5708" />
   </joint>
   <joint name="mid360_imu_joint" type="fixed">

Commit message: Updated urdf for v1

File: lunabot_description/urdf/v1_bot.urdf.xacro (robot description, xacro)
@@ -157,5 +157,5 @@
     <parent link="base_link" />
     <child link="camera_front_link" />
-    <origin xyz="0.40 0 0.54" rpy="0 0.523599 0" />
+    <origin xyz="0.62 0 0.35" rpy="0 0.523599 0" />
   </joint>
   <joint name="camera_front_optical_joint" type="fixed">
@@ -167,5 +167,5 @@
     <parent link="base_link" />
     <child link="camera_back_link" />
-    <origin xyz="-0.128 0 0.5" rpy="0 0.523599 3.14" />
+    <origin xyz="-0.02 0 0.58" rpy="0 0.523599 3.14" />
   </joint>
   <joint name="camera_back_optical_joint" type="fixed">
@@ -177,5 +177,5 @@
     <parent link="base_link" />
     <child link="livox_frame" />
-    <origin xyz="-0.128 0 0.46" rpy="3.14159 0 -1.5708" />
+    <origin xyz="0.032 0 0.54" rpy="3.14159 0 -1.5708" />
   </joint>
   <joint name="mid360_imu_joint" type="fixed">

Commit message: Modified urdf and image compressor

File: lunabot_description/urdf/v1_bot.urdf.xacro (robot description, xacro)
@@ -14,6 +14,6 @@
   </xacro:if>
   <xacro:unless value="$(arg use_sim)">
-    <xacro:property name="camera_sim_link_offset" value="0.15" />
-    <xacro:property name="camera_sim_joint_offset" value="0.15" />
+    <xacro:property name="camera_sim_link_offset" value="0" />
+    <xacro:property name="camera_sim_joint_offset" value="0" />
   </xacro:unless>
   <!-- ================================= -->
@@ -177,5 +177,5 @@
     <parent link="base_link" />
     <child link="livox_frame" />
-    <origin xyz="0.032 0 0.54" rpy="3.14159 0 -1.5708" />
+    <origin xyz="0.032 0 0.54" rpy="3.14159 0 1.5708" />
   </joint>
   <joint name="mid360_imu_joint" type="fixed">

Commit message: Modifying URDF

File: lunabot_description/urdf/v1_bot.urdf.xacro (robot description, xacro)
@@ -177,5 +177,5 @@
     <parent link="base_link" />
     <child link="livox_frame" />
-    <origin xyz="0.032 0 0.54" rpy="3.14159 0 1.5708" />
+    <origin xyz="0.032 0 0.54" rpy="3.14159 0 0" />
   </joint>
   <joint name="mid360_imu_joint" type="fixed">

Commit message: Fixed imu joint

File: lunabot_description/urdf/v1_bot.urdf.xacro (robot description, xacro)
@@ -182,5 +182,5 @@
     <parent link="base_link" />
     <child link="mid360_imu_link" />
-    <origin xyz="-0.128 0 0.46" rpy="0 0 0" />
+    <origin xyz="-0.128 0 0.46" rpy="3.14159 0 0" />
   </joint>
   <!-- ================================= -->

File: lunabot_description/urdf/v2_bot.urdf.xacro (robot description, xacro)
@@ -245,5 +245,5 @@
     <parent link="base_link" />
     <child link="livox_frame" />
-    <origin xyz="-0.27 0 0.548" rpy="3.14159 0 -1.5708" />
+    <origin xyz="-0.27 0 0.548" rpy="3.14159 0 0" />
   </joint>
   <joint name="mid360_imu_joint" type="fixed">

Commit message: Applied correct rotation to pointlio quaternion due to rotated lidar irl, modified gui style

File: lunabot_description/urdf/v1_bot.urdf.xacro (robot description, xacro)
@@ -177,10 +177,10 @@
     <parent link="base_link" />
     <child link="livox_frame" />
-    <origin xyz="0.032 0 0.54" rpy="3.14159 0 0" />
+    <origin xyz="0.032 0 0.54" rpy="3.14159 0 1.5708" />
   </joint>
   <joint name="mid360_imu_joint" type="fixed">
     <parent link="base_link" />
     <child link="mid360_imu_link" />
-    <origin xyz="-0.128 0 0.46" rpy="3.14159 0 0" />
+    <origin xyz="0.032 0 0.54" rpy="3.14159 0 1.5708" />
   </joint>
   <!-- ================================= -->

File: lunabot_description/urdf/v2_bot.urdf.xacro (robot description, xacro)
@@ -245,10 +245,10 @@
     <parent link="base_link" />
     <child link="livox_frame" />
-    <origin xyz="-0.27 0 0.548" rpy="3.14159 0 0" />
+    <origin xyz="-0.27 0 0.548" rpy="3.14159 0 1.5708" />
   </joint>
   <joint name="mid360_imu_joint" type="fixed">
     <parent link="base_link" />
     <child link="mid360_imu_link" />
-    <origin xyz="-0.27 0 0.548" rpy="3.14159 0 0" />
+    <origin xyz="-0.27 0 0.548" rpy="3.14159 0 1.5708" />
   </joint>
   <!-- ================================= -->

Commit message: Applied fisheye rotation fix, gui styling

File: lunabot_description/urdf/v1_bot.urdf.xacro (robot description, xacro)
@@ -80,4 +80,39 @@
   </link>
   <link name="camera_back_optical_link"></link>
+  <link name="camera_fisheye_mount_link">
+    <inertial>
+      <mass value="0.05" />
+      <origin xyz="0 0 0" />
+      <inertia ixx="0.00001" ixy="0.0" ixz="0.0" iyy="0.00001" iyz="0.0" izz="0.00001" />
+    </inertial>
+  </link>
+  <link name="camera_fisheye_yaw_link">
+    <inertial>
+      <mass value="0.05" />
+      <origin xyz="0 0 0" />
+      <inertia ixx="0.00001" ixy="0.0" ixz="0.0" iyy="0.00001" iyz="0.0" izz="0.00001" />
+    </inertial>
+  </link>
+  <link name="camera_fisheye_link">
+    <inertial>
+      <mass value="0.1" />
+      <origin xyz="0 0 0" />
+      <inertia ixx="0.0001" ixy="0.0" ixz="0.0" iyy="0.0001" iyz="0.0" izz="0.0001" />
+    </inertial>
+    <visual>
+      <geometry>
+        <mesh
+          filename="file:///$(find lunabot_description)/meshes/v2_bot/v2_bot_fisheye_camera.stl" />
+      </geometry>
+      <material name="camera_grey" />
+    </visual>
+    <collision>
+      <geometry>
+        <mesh
+          filename="file:///$(find lunabot_description)/meshes/v2_bot/v2_bot_fisheye_camera.stl" />
+      </geometry>
+    </collision>
+  </link>
+  <link name="camera_fisheye_optical_link"></link>
   <link name="livox_frame">
     <visual>
@@ -172,4 +207,27 @@
     <parent link="camera_back_link" />
     <child link="camera_back_optical_link" />
+    <origin xyz="0 0 0" rpy="-1.5708 0 -1.5708" />
+  </joint>
+  <joint name="base_camera_fisheye_mount_joint" type="fixed">
+    <parent link="base_link" />
+    <child link="camera_fisheye_mount_link" />
+    <origin xyz="0.032 0 0.556" rpy="0 0 0" />
+  </joint>
+  <joint name="camera_fisheye_yaw_joint" type="revolute">
+    <parent link="camera_fisheye_mount_link" />
+    <child link="camera_fisheye_yaw_link" />
+    <origin xyz="0 0 0" rpy="0 0 0" />
+    <axis xyz="0 0 1" />
+    <limit effort="10" velocity="1.0" lower="-3.14159" upper="3.14159" />
+    <dynamics damping="0.1" friction="0.1" />
+  </joint>
+  <joint name="camera_fisheye_pitch_joint" type="fixed">
+    <parent link="camera_fisheye_yaw_link" />
+    <child link="camera_fisheye_link" />
+    <origin xyz="0 0 0" rpy="0 0.523599 0" />
+  </joint>
+  <joint name="camera_fisheye_optical_joint" type="fixed">
+    <parent link="camera_fisheye_link" />
+    <child link="camera_fisheye_optical_link" />
     <origin xyz="0 0 0" rpy="-1.5708 0 -1.5708" />
   </joint>
@@ -345,4 +403,42 @@
           </ros>
           <frame_name>camera_back_optical_link</frame_name>
+          <publish_tf>false</publish_tf>
+          <publish_point_cloud>true</publish_point_cloud>
+        </plugin>
+      </sensor>
+      <material>Gazebo/Grey</material>
+    </gazebo>
+    <gazebo reference="camera_fisheye_link">
+      <sensor type="depth" name="camera_fisheye">
+        <pose>0 0 0 0 0 0</pose>
+        <update_rate>60.0</update_rate>
+        <visualize>false</visualize>
+        <camera>
+          <horizontal_fov>2.1</horizontal_fov>
+          <image>
+            <width>640</width>
+            <height>360</height>
+            <format>R8G8B8</format>
+          </image>
+          <distortion>
+            <k1>0.0</k1>
+            <k2>0.0</k2>
+            <k3>0.0</k3>
+            <p1>0.0</p1>
+            <p2>0.0</p2>
+          </distortion>
+          <clip>
+            <near>0.05</near>
+            <far>6.0</far>
+          </clip>
+        </camera>
+        <plugin name="camera_fisheye_controller" filename="libgazebo_ros_camera.so">
+          <ros>
+            <remapping>/camera_fisheye/image_raw:=/camera_fisheye/color/image_raw</remapping>
+            <remapping>/camera_fisheye/points:=/camera_fisheye/color/points</remapping>
+            <remapping>/camera_fisheye/camera_info:=/camera_fisheye/color/camera_info</remapping>
+            <remapping>/camera_fisheye/depth/image_raw:=/camera_fisheye/depth/image_rect_raw</remapping>
+          </ros>
+          <frame_name>camera_fisheye_optical_link</frame_name>
           <publish_tf>false</publish_tf>
           <publish_point_cloud>true</publish_point_cloud>
@@ -457,4 +553,14 @@
         <state_interface name="velocity" />
       </joint>
+      <joint name="camera_fisheye_yaw_joint">
+        <command_interface name="position">
+          <param name="min">-3.14159</param>
+          <param name="max">3.14159</param>
+        </command_interface>
+        <state_interface name="position">
+          <param name="initial_value">0.0</param>
+        </state_interface>
+        <state_interface name="velocity" />
+      </joint>
     </ros2_control>
   </xacro:if>

File: lunabot_description/urdf/v2_bot.urdf.xacro (robot description, xacro)
@@ -108,4 +108,11 @@
     </inertial>
   </link>
+  <link name="camera_fisheye_yaw_link">
+    <inertial>
+      <mass value="0.05" />
+      <origin xyz="0 0 0" />
+      <inertia ixx="0.00001" ixy="0.0" ixz="0.0" iyy="0.00001" iyz="0.0" izz="0.00001" />
+    </inertial>
+  </link>
   <link name="camera_fisheye_link">
     <inertial>
@@ -227,13 +234,18 @@
     <parent link="base_link" />
     <child link="camera_fisheye_mount_link" />
-    <origin xyz="-0.22 0 0.564" rpy="0 0.523599 0" />
+    <origin xyz="-0.22 0 0.564" rpy="0 0 0" />
   </joint>
   <joint name="camera_fisheye_yaw_joint" type="revolute">
     <parent link="camera_fisheye_mount_link" />
-    <child link="camera_fisheye_link" />
+    <child link="camera_fisheye_yaw_link" />
     <origin xyz="0 0 0" rpy="0 0 0" />
     <axis xyz="0 0 1" />
     <limit effort="10" velocity="1.0" lower="-3.14159" upper="3.14159" />
     <dynamics damping="0.1" friction="0.1" />
+  </joint>
+  <joint name="camera_fisheye_pitch_joint" type="fixed">
+    <parent link="camera_fisheye_yaw_link" />
+    <child link="camera_fisheye_link" />
+    <origin xyz="0 0 0" rpy="0 0.523599 0" />
   </joint>
   <joint name="camera_fisheye_optical_joint" type="fixed">

Commit message: Lined up sensors in v1, fixed fisheye rotation

File: lunabot_description/urdf/v1_bot.urdf.xacro (robot description, xacro)
@@ -10,10 +10,14 @@
   </material>
   <xacro:if value="$(arg use_sim)">
-    <xacro:property name="camera_sim_link_offset" value="0.015" />
+    <xacro:property name="camera_sim_link_offset" value="-0.01" />
     <xacro:property name="camera_sim_joint_offset" value="0" />
+    <xacro:property name="lidar_sim_link_offset" value="0.01" />
+    <xacro:property name="lidar_sim_joint_offset" value="0" />
   </xacro:if>
   <xacro:unless value="$(arg use_sim)">
     <xacro:property name="camera_sim_link_offset" value="0" />
     <xacro:property name="camera_sim_joint_offset" value="0" />
+    <xacro:property name="lidar_sim_link_offset" value="0" />
+    <xacro:property name="lidar_sim_joint_offset" value="0" />
   </xacro:unless>
   <!-- ================================= -->
@@ -50,5 +54,5 @@
           filename="file:///$(find lunabot_description)/meshes/v1_bot/v1_bot_d456_camera.stl" />
       </geometry>
-      <origin xyz="0 -${camera_sim_link_offset} 0" rpy="0 0 0" />
+      <origin xyz="0 ${camera_sim_link_offset} 0" rpy="0 0 0" />
       <material name="camera_grey" />
     </visual>
@@ -58,5 +62,5 @@
           filename="file:///$(find lunabot_description)/meshes/v1_bot/v1_bot_d456_camera.stl" />
       </geometry>
-      <origin xyz="0 -${camera_sim_link_offset} 0" rpy="0 0 0" />
+      <origin xyz="0 ${camera_sim_link_offset} 0" rpy="0 0 0" />
     </collision>
   </link>
@@ -68,5 +72,5 @@
           filename="file:///$(find lunabot_description)/meshes/v1_bot/v1_bot_d456_camera.stl" />
       </geometry>
-      <origin xyz="0 -${camera_sim_link_offset} 0" rpy="0 0 0" />
+      <origin xyz="0 ${camera_sim_link_offset} 0" rpy="0 0 0" />
       <material name="camera_grey" />
     </visual>
@@ -76,5 +80,5 @@
           filename="file:///$(find lunabot_description)/meshes/v1_bot/v1_bot_d456_camera.stl" />
       </geometry>
-      <origin xyz="0 -${camera_sim_link_offset} 0" rpy="0 0 0" />
+      <origin xyz="0 ${camera_sim_link_offset} 0" rpy="0 0 0" />
     </collision>
   </link>
@@ -90,7 +94,21 @@
     <inertial>
       <mass value="0.05" />
-      <origin xyz="0 0 0" />
+      <origin xyz="0.035 0 0" rpy="0 0 1.5708" />
       <inertia ixx="0.00001" ixy="0.0" ixz="0.0" iyy="0.00001" iyz="0.0" izz="0.00001" />
     </inertial>
+    <visual>
+      <geometry>
+        <mesh
+          filename="file:///$(find lunabot_description)/meshes/v1_bot/v1_bot_fisheye_mount.dae" />
+      </geometry>
+      <origin xyz="0.035 0 0" rpy="0 0 1.5708" />
+      <material name="camera_grey" />
+    </visual>
+    <collision>
+      <geometry>
+        <mesh
+          filename="file:///$(find lunabot_description)/meshes/v1_bot/v1_bot_fisheye_mount.stl" />
+      </geometry>
+    </collision>
   </link>
   <link name="camera_fisheye_link">
@@ -103,5 +121,5 @@
       <geometry>
         <mesh
-          filename="file:///$(find lunabot_description)/meshes/v2_bot/v2_bot_fisheye_camera.stl" />
+          filename="file:///$(find lunabot_description)/meshes/v1_bot/v1_bot_fisheye_camera.stl" />
       </geometry>
       <material name="camera_grey" />
@@ -110,5 +128,5 @@
       <geometry>
         <mesh
-          filename="file:///$(find lunabot_description)/meshes/v2_bot/v2_bot_fisheye_camera.stl" />
+          filename="file:///$(find lunabot_description)/meshes/v1_bot/v1_bot_fisheye_camera.stl" />
       </geometry>
     </collision>
@@ -119,6 +137,7 @@
       <geometry>
         <mesh
-          filename="file:///$(find lunabot_description)/meshes/v1_bot/v1_bot_mid360_lidar.stl" />
-      </geometry>
+          filename="file:///$(find lunabot_description)/meshes/v1_bot/v1_bot_mid360_lidar.dae" />
+      </geometry>
+      <origin xyz="${lidar_sim_link_offset} 0 0" rpy="0 0 0" />
       <material name="camera_grey" />
     </visual>
@@ -128,4 +147,5 @@
           filename="file:///$(find lunabot_description)/meshes/v1_bot/v1_bot_mid360_lidar.stl" />
       </geometry>
+      <origin xyz="${lidar_sim_link_offset} 0 0" rpy="0 0 0" />
     </collision>
   </link>
@@ -141,5 +161,5 @@
     </inertial>
     <collision>
-      <geometry>
+      <geometry>xacro
         <cylinder length="0.127" radius="0.1016" />
       </geometry>
@@ -192,5 +212,5 @@
     <parent link="base_link" />
     <child link="camera_front_link" />
-    <origin xyz="0.62 0 0.35" rpy="0 0.523599 0" />
+    <origin xyz="0.526 0 0.584" rpy="0 0.785398 0" />
   </joint>
   <joint name="camera_front_optical_joint" type="fixed">
@@ -202,5 +222,5 @@
     <parent link="base_link" />
     <child link="camera_back_link" />
-    <origin xyz="-0.02 0 0.58" rpy="0 0.523599 3.14" />
+    <origin xyz="-0.277 0 0.602" rpy="0 0.785398 3.14" />
   </joint>
   <joint name="camera_back_optical_joint" type="fixed">
@@ -212,10 +232,10 @@
     <parent link="base_link" />
     <child link="camera_fisheye_mount_link" />
-    <origin xyz="0.032 0 0.556" rpy="0 0 0" />
+    <origin xyz="-0.2 0 0.635" rpy="0 0 0" />
   </joint>
   <joint name="camera_fisheye_yaw_joint" type="revolute">
     <parent link="camera_fisheye_mount_link" />
     <child link="camera_fisheye_yaw_link" />
-    <origin xyz="0 0 0" rpy="0 0 0" />
+    <origin xyz="-0.035 0 0" rpy="0 0 0" />
     <axis xyz="0 0 1" />
     <limit effort="10" velocity="1.0" lower="-3.14159" upper="3.14159" />
@@ -225,5 +245,5 @@
     <parent link="camera_fisheye_yaw_link" />
     <child link="camera_fisheye_link" />
-    <origin xyz="0 0 0" rpy="0 0.523599 0" />
+    <origin xyz="0.077 0 -0.006" rpy="0 0.785398 0" />
   </joint>
   <joint name="camera_fisheye_optical_joint" type="fixed">
@@ -235,10 +255,10 @@
     <parent link="base_link" />
     <child link="livox_frame" />
-    <origin xyz="0.032 0 0.54" rpy="3.14159 0 1.5708" />
+    <origin xyz="-0.23 0 0.59" rpy="3.14159 0 1.5708" />
   </joint>
   <joint name="mid360_imu_joint" type="fixed">
     <parent link="base_link" />
     <child link="mid360_imu_link" />
-    <origin xyz="0.032 0 0.54" rpy="3.14159 0 1.5708" />
+    <origin xyz="-0.23 0 0.59" rpy="3.14159 0 1.5708" />
   </joint>
   <!-- ================================= -->
@@ -273,4 +293,8 @@
   <!-- ================================= -->
   <xacro:if value="$(arg use_sim)">
+    <gazebo reference="base_link">
+    </gazebo>
+    <gazebo reference="camera_fisheye_yaw_link">
+    </gazebo>
     <gazebo reference="front_right_wheel_link">
       <material>Gazebo/Grey</material>

File: lunabot_description/urdf/v2_bot.urdf.xacro (robot description, xacro)
@@ -114,4 +114,17 @@
       <inertia ixx="0.00001" ixy="0.0" ixz="0.0" iyy="0.00001" iyz="0.0" izz="0.00001" />
     </inertial>
+    <visual>
+      <geometry>
+        <mesh
+          filename="file:///$(find lunabot_description)/meshes/v2_bot/v2_bot_fisheye_mount.dae" />
+      </geometry>
+      <material name="camera_grey" />
+    </visual>
+    <collision>
+      <geometry>
+        <mesh
+          filename="file:///$(find lunabot_description)/meshes/v2_bot/v2_bot_fisheye_mount.stl" />
+      </geometry>
+    </collision>
   </link>
   <link name="camera_fisheye_link">
@@ -247,5 +260,5 @@
     <parent link="camera_fisheye_yaw_link" />
     <child link="camera_fisheye_link" />
-    <origin xyz="0 0 0" rpy="0 0.523599 0" />
+    <origin xyz="0.07 0 0.035" rpy="0 0.523599 0" />
   </joint>
   <joint name="camera_fisheye_optical_joint" type="fixed">
@@ -306,4 +319,8 @@
   <!-- ================================= -->
   <xacro:if value="$(arg use_sim)">
+    <gazebo reference="base_link">
+    </gazebo>
+    <gazebo reference="camera_fisheye_yaw_link">
+    </gazebo>
     <gazebo reference="front_right_wheel_link">
       <material>Gazebo/Grey</material>

Commit message: Updated to be compatible with ros2 jazzy

File: lunabot_description/urdf/v1_bot.urdf.xacro (robot description, xacro)
@@ -3,4 +3,12 @@
   xmlns:xacro="http://www.ros.org/wiki/xacro">
   <xacro:arg name="use_sim" default="true" />
+  <xacro:if value="$(arg use_sim)">
+    <xacro:property name="camera_sim_link_offset" value="-0.01" />
+    <xacro:property name="lidar_sim_link_offset" value="0.01" />
+  </xacro:if>
+  <xacro:unless value="$(arg use_sim)">
+    <xacro:property name="camera_sim_link_offset" value="0" />
+    <xacro:property name="lidar_sim_link_offset" value="0" />
+  </xacro:unless>
   <material name="camera_grey">
     <color rgba="0.81 0.81 0.81 1.0" />
@@ -9,16 +17,4 @@
     <color rgba="0.22 0.22 0.22 1.0" />
   </material>
-  <xacro:if value="$(arg use_sim)">
-    <xacro:property name="camera_sim_link_offset" value="-0.01" />
-    <xacro:property name="camera_sim_joint_offset" value="0" />
-    <xacro:property name="lidar_sim_link_offset" value="0.01" />
-    <xacro:property name="lidar_sim_joint_offset" value="0" />
-  </xacro:if>
-  <xacro:unless value="$(arg use_sim)">
-    <xacro:property name="camera_sim_link_offset" value="0" />
-    <xacro:property name="camera_sim_joint_offset" value="0" />
-    <xacro:property name="lidar_sim_link_offset" value="0" />
-    <xacro:property name="lidar_sim_joint_offset" value="0" />
-  </xacro:unless>
   <!-- ================================= -->
   <!--            BODY LINKS             -->

File: lunabot_description/urdf/v2_bot.urdf.xacro (robot description, xacro)
@@ -3,4 +3,10 @@
   xmlns:xacro="http://www.ros.org/wiki/xacro">
   <xacro:arg name="use_sim" default="true" />
+  <xacro:if value="$(arg use_sim)">
+    <xacro:property name="camera_sim_link_offset" value="0.01" />
+  </xacro:if>
+  <xacro:unless value="$(arg use_sim)">
+    <xacro:property name="camera_sim_link_offset" value="0" />
+  </xacro:unless>
   <material name="camera_grey">
     <color rgba="0.81 0.81 0.81 1.0" />
@@ -9,12 +15,4 @@
     <color rgba="0.22 0.22 0.22 1.0" />
   </material>
-  <xacro:if value="$(arg use_sim)">
-    <xacro:property name="camera_sim_link_offset" value="0.01" />
-    <xacro:property name="camera_sim_joint_offset" value="0" />
-  </xacro:if>
-  <xacro:unless value="$(arg use_sim)">
-    <xacro:property name="camera_sim_link_offset" value="0" />
-    <xacro:property name="camera_sim_joint_offset" value="0" />
-  </xacro:unless>
   <!-- ================================= -->
   <!--            BODY LINKS             -->
