Commit message: using base footprint to correct height
Co-authored-by: Copilot <copilot@github.com>

File: lunabot_description/urdf/v2_bot.urdf.xacro (robot description, xacro)
@@ -18,4 +18,10 @@
   <!--            BODY LINKS             -->
   <!-- ================================= -->
+  <link name="base_footprint"></link>
+  <joint name="base_footprint_joint" type="fixed">
+    <parent link="base_footprint" />
+    <child link="base_link" />
+    <origin xyz="0 0 -0.3556" rpy="0 0 0" />
+  </joint>
   <link name="base_link">
     <visual>
@@ -45,5 +51,6 @@
           filename="file:///$(find lunabot_description)/meshes/v2_bot/v2_bot_bucket.stl" />
       </geometry>
-      <origin xyz="0.2 0 0" rpy="1.5708 0 1.5708" />
+      <origin xyz="0.2 0 0" rpy="0 0 1.5708" />
+      <material name="camera_grey" />
     </visual>
     <!-- <collision>
@@ -225,5 +232,5 @@
     <parent link="base_link" />
     <child link="camera_front_link" />
-    <origin xyz="0.55 0 0.425" rpy="0 0.523599 0" />
+    <origin xyz="0.55 0 0.425" rpy="0 0.785398 0" />
   </joint>
   <joint name="camera_front_optical_joint" type="fixed">

Commit message: Updated v2 robot model, reverted base_footprint
Co-authored-by: Copilot <copilot@github.com>

File: lunabot_description/urdf/v2_bot.urdf.xacro (robot description, xacro)
@@ -7,5 +7,5 @@
   </xacro:if>
   <xacro:unless value="$(arg use_sim)">
-    <xacro:property name="camera_sim_link_offset" value="0" />
+    <xacro:property name="camera_sim_link_offset" value="0.019" />
   </xacro:unless>
   <material name="camera_grey">
@@ -18,10 +18,4 @@
   <!--            BODY LINKS             -->
   <!-- ================================= -->
-  <link name="base_footprint"></link>
-  <joint name="base_footprint_joint" type="fixed">
-    <parent link="base_footprint" />
-    <child link="base_link" />
-    <origin xyz="0 0 -0.3556" rpy="0 0 0" />
-  </joint>
   <link name="base_link">
     <visual>
@@ -30,5 +24,5 @@
           filename="file:///$(find lunabot_description)/meshes/v2_bot/v2_bot_body.dae" />
       </geometry>
-      <origin xyz="0 0 0.1625" rpy="0 0 1.5708" />
+      <origin xyz="0 -0.008 0.1625" rpy="0 0 1.5708" />
     </visual>
     <collision>
@@ -54,5 +48,5 @@
       <material name="camera_grey" />
     </visual>
-    <!-- <collision>
+    <collision>
       <geometry>
         <mesh
@@ -60,5 +54,5 @@
       </geometry>
       <origin xyz="0.2 0 0" rpy="1.5708 0 1.5708" />
-    </collision> -->
+    </collision>
     <inertial>
       <mass value="3.0" />
@@ -125,4 +119,5 @@
       </geometry>
       <material name="camera_grey" />
+      <origin xyz="0 0 0" rpy="0 0 -1.5708" />
     </visual>
     <collision>
@@ -131,4 +126,5 @@
           filename="file:///$(find lunabot_description)/meshes/v2_bot/v2_bot_fisheye_mount.stl" />
       </geometry>
+      <origin xyz="0 0 0" rpy="0 0 -1.5708" />
     </collision>
   </link>
@@ -144,5 +140,6 @@
           filename="file:///$(find lunabot_description)/meshes/v2_bot/v2_bot_fisheye_camera.stl" />
       </geometry>
-      <material name="camera_grey" />
+      <origin xyz="0 0 0" rpy="0 0 3.14" />
+      <material name="black" />
     </visual>
         <collision>
@@ -151,5 +148,6 @@
           filename="file:///$(find lunabot_description)/meshes/v2_bot/v2_bot_fisheye_camera.stl" />
       </geometry>
-      <material name="camera_grey" />
+      <material name="black" />
+      <origin xyz="0 0 0" rpy="0 0 3.14" />
     </collision>
   </link>
@@ -232,5 +230,5 @@
     <parent link="base_link" />
     <child link="camera_front_link" />
-    <origin xyz="0.55 0 0.425" rpy="0 0.785398 0" />
+    <origin xyz="0.55 0 0.412" rpy="0 0.837758 0" />
   </joint>
   <joint name="camera_front_optical_joint" type="fixed">
@@ -242,5 +240,5 @@
     <parent link="base_link" />
     <child link="camera_back_link" />
-    <origin xyz="-0.324 0 0.564" rpy="0 0.785398 3.14" />
+    <origin xyz="-0.348 0 0.548" rpy="0 0.837758 3.14" />
   </joint>
   <joint name="camera_back_optical_joint" type="fixed">
@@ -252,5 +250,5 @@
     <parent link="base_link" />
     <child link="camera_fisheye_mount_link" />
-    <origin xyz="-0.22 0 0.564" rpy="0 0 0" />
+    <origin xyz="-0.34 -0.01 0.58" rpy="0 0 0" />
   </joint>
   <joint name="camera_fisheye_yaw_joint" type="revolute">
@@ -259,5 +257,5 @@
     <origin xyz="0 0 0" rpy="0 0 0" />
     <axis xyz="0 0 1" />
-    <limit effort="10" velocity="1.0" lower="-3.14159" upper="3.14159" />
+    <limit effort="10" velocity="1.0" lower="-1.5708" upper="1.5708" />
     <dynamics damping="0.1" friction="0.1" />
   </joint>
@@ -265,5 +263,5 @@
     <parent link="camera_fisheye_yaw_link" />
     <child link="camera_fisheye_link" />
-    <origin xyz="0.07 0 0.035" rpy="0 0.523599 0" />
+    <origin xyz="-0.045 0 -0.005" rpy="0 -0.785398 0" />
   </joint>
   <joint name="camera_fisheye_optical_joint" type="fixed">
@@ -275,10 +273,10 @@
     <parent link="base_link" />
     <child link="livox_frame" />
-    <origin xyz="-0.27 0 0.548" rpy="3.14159 0 1.5708" />
+    <origin xyz="-0.3 0 0.548" rpy="3.14159 0 1.5708" />
   </joint>
   <joint name="mid360_imu_joint" type="fixed">
     <parent link="base_link" />
     <child link="mid360_imu_link" />
-    <origin xyz="-0.27 0 0.548" rpy="3.14159 0 1.5708" />
+    <origin xyz="-0.3 0 0.548" rpy="3.14159 0 1.5708" />
   </joint>
   <!-- ================================= -->
@@ -288,5 +286,5 @@
     <parent link="base_link" />
     <child link="bucket_link" />
-    <origin xyz="-0.15 0 0.2" rpy="0 0 0" />
+    <origin xyz="-0.204 0 0.162" rpy="0 0 0" />
     <axis xyz="0 1 0" />
     <limit effort="100" velocity="0.3" lower="-1.57" upper="0.1" />
@@ -620,6 +618,6 @@
       <joint name="camera_fisheye_yaw_joint">
         <command_interface name="position">
-          <param name="min">-3.14159</param>
-          <param name="max">3.14159</param>
+          <param name="min">-1.5708</param>
+          <param name="max">1.5708</param>
         </command_interface>
         <state_interface name="position">
