Commit message: Initial gui setup

File: lunabot_description/urdf/v2_bot.urdf.xacro (robot description, xacro)
@@ -101,4 +101,33 @@
   </link>
   <link name="camera_back_optical_link"></link>
+  <link name="camera_fisheye_mount_link">
+    <inertial>
+      <mass value="0.05" />
+      <origin xyz="0 0 0" />
+      <inertia ixx="0.00001" ixy="0.0" ixz="0.0" iyy="0.00001" iyz="0.0" izz="0.00001" />
+    </inertial>
+  </link>
+  <link name="camera_fisheye_link">
+    <inertial>
+      <mass value="0.1" />
+      <origin xyz="0 0 0" />
+      <inertia ixx="0.0001" ixy="0.0" ixz="0.0" iyy="0.0001" iyz="0.0" izz="0.0001" />
+    </inertial>
+    <visual>
+      <geometry>
+        <mesh
+          filename="file:///$(find lunabot_description)/meshes/v2_bot/v2_bot_fisheye_camera.stl" />
+      </geometry>
+      <material name="camera_grey" />
+    </visual>
+        <collision>
+      <geometry>
+        <mesh
+          filename="file:///$(find lunabot_description)/meshes/v2_bot/v2_bot_fisheye_camera.stl" />
+      </geometry>
+      <material name="camera_grey" />
+    </collision>
+  </link>
+  <link name="camera_fisheye_optical_link"></link>
   <link name="mid360_lidar_link">
     <visual>
@@ -193,4 +222,22 @@
     <parent link="camera_back_link" />
     <child link="camera_back_optical_link" />
+    <origin xyz="0 0 0" rpy="-1.5708 0 -1.5708" />
+  </joint>
+  <joint name="base_camera_fisheye_mount_joint" type="fixed">
+    <parent link="base_link" />
+    <child link="camera_fisheye_mount_link" />
+    <origin xyz="-0.22 0 0.564" rpy="0 0.523599 0" />
+  </joint>
+  <joint name="camera_fisheye_yaw_joint" type="revolute">
+    <parent link="camera_fisheye_mount_link" />
+    <child link="camera_fisheye_link" />
+    <origin xyz="0 0 0" rpy="0 0 0" />
+    <axis xyz="0 0 1" />
+    <limit effort="10" velocity="1.0" lower="-3.14159" upper="3.14159" />
+    <dynamics damping="0.1" friction="0.1" />
+  </joint>
+  <joint name="camera_fisheye_optical_joint" type="fixed">
+    <parent link="camera_fisheye_link" />
+    <child link="camera_fisheye_optical_link" />
     <origin xyz="0 0 0" rpy="-1.5708 0 -1.5708" />
   </joint>
@@ -328,5 +375,5 @@
           <clip>
             <near>0.05</near>
-            <far>10.0</far>
+            <far>6.0</far>
           </clip>
         </camera>
@@ -366,5 +413,5 @@
           <clip>
             <near>0.05</near>
-            <far>10.0</far>
+            <far>6.0</far>
           </clip>
         </camera>
@@ -377,4 +424,42 @@
           </ros>
           <frame_name>camera_back_optical_link</frame_name>
+          <publish_tf>false</publish_tf>
+          <publish_point_cloud>true</publish_point_cloud>
+        </plugin>
+      </sensor>
+      <material>Gazebo/Grey</material>
+    </gazebo>
+    <gazebo reference="camera_fisheye_link">
+      <sensor type="depth" name="camera_fisheye">
+        <pose>0 0 0 0 0 0</pose>
+        <update_rate>60.0</update_rate>
+        <visualize>false</visualize>
+        <camera>
+          <horizontal_fov>2.1</horizontal_fov>
+          <image>
+            <width>640</width>
+            <height>360</height>
+            <format>R8G8B8</format>
+          </image>
+          <distortion>
+            <k1>0.0</k1>
+            <k2>0.0</k2>
+            <k3>0.0</k3>
+            <p1>0.0</p1>
+            <p2>0.0</p2>
+          </distortion>
+          <clip>
+            <near>0.05</near>
+            <far>6.0</far>
+          </clip>
+        </camera>
+        <plugin name="camera_fisheye_controller" filename="libgazebo_ros_camera.so">
+          <ros>
+            <remapping>/camera_fisheye/image_raw:=/camera_fisheye/color/image_raw</remapping>
+            <remapping>/camera_fisheye/points:=/camera_fisheye/color/points</remapping>
+            <remapping>/camera_fisheye/camera_info:=/camera_fisheye/color/camera_info</remapping>
+            <remapping>/camera_fisheye/depth/image_raw:=/camera_fisheye/depth/image_rect_raw</remapping>
+          </ros>
+          <frame_name>camera_fisheye_optical_link</frame_name>
           <publish_tf>false</publish_tf>
           <publish_point_cloud>true</publish_point_cloud>
@@ -499,4 +584,14 @@
         <state_interface name="velocity" />
       </joint>
+      <joint name="camera_fisheye_yaw_joint">
+        <command_interface name="position">
+          <param name="min">-3.14159</param>
+          <param name="max">3.14159</param>
+        </command_interface>
+        <state_interface name="position">
+          <param name="initial_value">0.0</param>
+        </state_interface>
+        <state_interface name="velocity" />
+      </joint>
     </ros2_control>
   </xacro:if>

Commit message: Tuned rtabmap in sim on humble, added lidar to rtabmap, added livox msg to pointcloud converter node, fixed some gui issues

File: lunabot_description/urdf/v2_bot.urdf.xacro (robot description, xacro)
@@ -48,5 +48,5 @@
       <material name="camera_grey" />
     </visual>
-    <collision>
+    <!-- <collision>
       <geometry>
         <mesh
@@ -54,5 +54,5 @@
       </geometry>
       <origin xyz="0.2 0 0" rpy="1.5708 0 1.5708" />
-    </collision>
+    </collision> -->
     <inertial>
       <mass value="3.0" />
@@ -612,5 +612,5 @@
         </command_interface>
         <state_interface name="position">
-          <param name="initial_value">-0.2</param>
+          <param name="initial_value">0.0</param>
         </state_interface>
         <state_interface name="velocity" />
