Commit message: Remove leftover 90 deg CW rotation hack, remove points from inside robot boundary, fix sim fisheye and compression, added lidar to rtabmap

File: lunabot_description/urdf/v2_bot.urdf.xacro (robot description, xacro)
@@ -119,5 +119,5 @@
       </geometry>
       <material name="camera_grey" />
-      <origin xyz="0 0 0" rpy="0 0 -1.5708" />
+      <origin xyz="0 0 0" rpy="0 0 1.5708" />
     </visual>
     <collision>
@@ -126,5 +126,5 @@
           filename="file:///$(find lunabot_description)/meshes/v2_bot/v2_bot_fisheye_mount.stl" />
       </geometry>
-      <origin xyz="0 0 0" rpy="0 0 -1.5708" />
+      <origin xyz="0 0 0" rpy="0 0 1.5708" />
     </collision>
   </link>
@@ -255,7 +255,7 @@
     <parent link="camera_fisheye_mount_link" />
     <child link="camera_fisheye_yaw_link" />
-    <origin xyz="0 0 0" rpy="0 0 0" />
+    <origin xyz="0 0 0" rpy="0 0 3.1416" />
     <axis xyz="0 0 1" />
-    <limit effort="10" velocity="1.0" lower="-1.5708" upper="1.5708" />
+    <limit effort="10" velocity="1.0" lower="-3.1416" upper="3.1416" />
     <dynamics damping="0.1" friction="0.1" />
   </joint>
@@ -263,5 +263,5 @@
     <parent link="camera_fisheye_yaw_link" />
     <child link="camera_fisheye_link" />
-    <origin xyz="-0.045 0 -0.005" rpy="0 -0.785398 0" />
+    <origin xyz="-0.045 0 -0.005" rpy="0 0.785398 0" />
   </joint>
   <joint name="camera_fisheye_optical_joint" type="fixed">
@@ -482,5 +482,5 @@
           </distortion>
           <clip>
-            <near>0.05</near>
+            <near>0.15</near>
             <far>6.0</far>
           </clip>

Commit message: Fix urdf and fast_lio frame id

File: lunabot_description/urdf/v2_bot.urdf.xacro (robot description, xacro)
@@ -9,4 +9,5 @@
     <xacro:property name="camera_sim_link_offset" value="0.019" />
   </xacro:unless>
+  <xacro:property name="sensor_plate_pitch" value="0.0873" />
   <material name="camera_grey">
     <color rgba="0.81 0.81 0.81 1.0" />
@@ -88,5 +89,5 @@
           filename="file:///$(find lunabot_description)/meshes/v2_bot/v2_bot_d456_camera.stl" />
       </geometry>
-      <origin xyz="0 -${camera_sim_link_offset} 0" rpy="0 0 0" />
+      <origin xyz="0 ${-camera_sim_link_offset - 0.08} 0" rpy="0 0 0" />  <!-- model drawn on the lidar centreline; the frame itself is offset -->
       <material name="camera_grey" />
     </visual>
@@ -96,5 +97,5 @@
           filename="file:///$(find lunabot_description)/meshes/v2_bot/v2_bot_d456_camera.stl" />
       </geometry>
-      <origin xyz="0 -${camera_sim_link_offset} 0" rpy="0 0 0" />
+      <origin xyz="0 ${-camera_sim_link_offset - 0.08} 0" rpy="0 0 0" />  <!-- model drawn on the lidar centreline; the frame itself is offset -->
     </collision>
   </link>
@@ -119,5 +120,5 @@
       </geometry>
       <material name="camera_grey" />
-      <origin xyz="0 0 0" rpy="0 0 1.5708" />
+      <origin xyz="0 -0.01 0" rpy="0 0 -1.5708" />
     </visual>
     <collision>
@@ -126,5 +127,5 @@
           filename="file:///$(find lunabot_description)/meshes/v2_bot/v2_bot_fisheye_mount.stl" />
       </geometry>
-      <origin xyz="0 0 0" rpy="0 0 1.5708" />
+      <origin xyz="0 -0.01 0" rpy="0 0 -1.5708" />
     </collision>
   </link>
@@ -140,5 +141,5 @@
           filename="file:///$(find lunabot_description)/meshes/v2_bot/v2_bot_fisheye_camera.stl" />
       </geometry>
-      <origin xyz="0 0 0" rpy="0 0 3.14" />
+      <origin xyz="0 0.01 0" rpy="0 0 0" />
       <material name="black" />
     </visual>
@@ -149,5 +150,5 @@
       </geometry>
       <material name="black" />
-      <origin xyz="0 0 0" rpy="0 0 3.14" />
+      <origin xyz="0 0.01 0" rpy="0 0 0" />
     </collision>
   </link>
@@ -159,4 +160,5 @@
           filename="file:///$(find lunabot_description)/meshes/v2_bot/v2_bot_mid360_lidar.dae" />
       </geometry>
+      <origin xyz="0.02 0 0" rpy="0 0 0" />  <!-- model nudged 2 cm to robot -y to match the base mesh -->
       <material name="camera_grey" />
     </visual>
@@ -166,7 +168,9 @@
           filename="file:///$(find lunabot_description)/meshes/v2_bot/v2_bot_mid360_lidar.stl" />
       </geometry>
+      <origin xyz="0.02 0 0" rpy="0 0 0" />
     </collision>
   </link>
   <link name="mid360_imu_link"></link>
+  <link name="sensor_plate_link"></link>
   <!-- ================================= -->
   <!--            WHEEL LINKS            -->
@@ -238,7 +242,7 @@
   </joint>
   <joint name="base_camera_back_joint" type="fixed">
-    <parent link="base_link" />
+    <parent link="sensor_plate_link" />
     <child link="camera_back_link" />
-    <origin xyz="-0.348 0 0.548" rpy="0 0.837758 3.14" />
+    <origin xyz="-0.048 -0.1 0" rpy="0 0.837758 3.14" />
   </joint>
   <joint name="camera_back_optical_joint" type="fixed">
@@ -250,10 +254,10 @@
     <parent link="base_link" />
     <child link="camera_fisheye_mount_link" />
-    <origin xyz="-0.34 -0.01 0.58" rpy="0 0 0" />
+    <origin xyz="-0.34 0.0 0.58" rpy="0 0 0" />
   </joint>
   <joint name="camera_fisheye_yaw_joint" type="revolute">
     <parent link="camera_fisheye_mount_link" />
     <child link="camera_fisheye_yaw_link" />
-    <origin xyz="0 0 0" rpy="0 0 3.1416" />
+    <origin xyz="0 0 0" rpy="0 0 0" />
     <axis xyz="0 0 1" />
     <limit effort="10" velocity="1.0" lower="-3.1416" upper="3.1416" />
@@ -263,5 +267,5 @@
     <parent link="camera_fisheye_yaw_link" />
     <child link="camera_fisheye_link" />
-    <origin xyz="-0.045 0 -0.005" rpy="0 0.785398 0" />
+    <origin xyz="-0.045 0 -0.005" rpy="0 0.785398 3.14159" />
   </joint>
   <joint name="camera_fisheye_optical_joint" type="fixed">
@@ -270,13 +274,18 @@
     <origin xyz="0 0 0" rpy="-1.5708 0 -1.5708" />
   </joint>
+  <joint name="base_sensor_plate_joint" type="fixed">
+    <parent link="base_link" />
+    <child link="sensor_plate_link" />
+    <origin xyz="-0.3 0 0.548" rpy="0 ${sensor_plate_pitch} 0" />
+  </joint>
   <joint name="base_mid360_joint" type="fixed">
-    <parent link="base_link" />
+    <parent link="sensor_plate_link" />
     <child link="livox_frame" />
-    <origin xyz="-0.3 0 0.548" rpy="3.14159 0 1.5708" />
+    <origin xyz="0 0 0" rpy="3.14159 0 -1.5708" />
   </joint>
   <joint name="mid360_imu_joint" type="fixed">
-    <parent link="base_link" />
+    <parent link="sensor_plate_link" />
     <child link="mid360_imu_link" />
-    <origin xyz="-0.3 0 0.548" rpy="3.14159 0 1.5708" />
+    <origin xyz="0 0 0" rpy="3.14159 0 -1.5708" />
   </joint>
   <!-- ================================= -->

Commit message: Flip base_link to the lidar side, rebuild UCF sim arena from the guidebook, fix sim wheel friction

File: lunabot_description/urdf/v2_bot.urdf.xacro (robot description, xacro)
@@ -19,5 +19,12 @@
   <!--            BODY LINKS             -->
   <!-- ================================= -->
-  <link name="base_link">
+  <!-- base_link +x is the driving front (lidar end), the chassis model has the bucket end at +x -->
+  <link name="base_link"></link>
+  <joint name="base_chassis_joint" type="fixed">
+    <parent link="base_link" />
+    <child link="chassis_link" />
+    <origin xyz="0 0 0" rpy="0 0 3.14159" />
+  </joint>
+  <link name="chassis_link">
     <visual>
       <geometry>
@@ -232,5 +239,5 @@
   <!-- ================================= -->
   <joint name="base_camera_front_joint" type="fixed">
-    <parent link="base_link" />
+    <parent link="chassis_link" />
     <child link="camera_front_link" />
     <origin xyz="0.55 0 0.412" rpy="0 0.837758 0" />
@@ -252,5 +259,5 @@
   </joint>
   <joint name="base_camera_fisheye_mount_joint" type="fixed">
-    <parent link="base_link" />
+    <parent link="chassis_link" />
     <child link="camera_fisheye_mount_link" />
     <origin xyz="-0.34 0.0 0.58" rpy="0 0 0" />
@@ -275,5 +282,5 @@
   </joint>
   <joint name="base_sensor_plate_joint" type="fixed">
-    <parent link="base_link" />
+    <parent link="chassis_link" />
     <child link="sensor_plate_link" />
     <origin xyz="-0.3 0 0.548" rpy="0 ${sensor_plate_pitch} 0" />
@@ -293,5 +300,5 @@
   <!-- ================================= -->
   <joint name="base_bucket_joint" type="revolute">
-    <parent link="base_link" />
+    <parent link="chassis_link" />
     <child link="bucket_link" />
     <origin xyz="-0.204 0 0.162" rpy="0 0 0" />
@@ -304,5 +311,5 @@
   <!-- ================================= -->
   <joint name="base_rear_right_wheel_joint" type="continuous">
-    <parent link="base_link" />
+    <parent link="chassis_link" />
     <child link="rear_right_wheel_link" />
     <origin xyz="-0.235 -0.25 0.08" rpy="0 0 0" />
@@ -310,5 +317,5 @@
   </joint>
   <joint name="base_rear_left_wheel_joint" type="continuous">
-    <parent link="base_link" />
+    <parent link="chassis_link" />
     <child link="rear_left_wheel_link" />
     <origin xyz="-0.235 0.25 0.08" rpy="0 0 0" />
@@ -316,5 +323,5 @@
   </joint>
   <joint name="base_front_right_wheel_joint" type="continuous">
-    <parent link="base_link" />
+    <parent link="chassis_link" />
     <child link="front_right_wheel_link" />
     <origin xyz="0.215 -0.25 0.08" rpy="0 0 0" />
@@ -322,5 +329,5 @@
   </joint>
   <joint name="base_front_left_wheel_joint" type="continuous">
-    <parent link="base_link" />
+    <parent link="chassis_link" />
     <child link="front_left_wheel_link" />
     <origin xyz="0.215 0.25 0.08" rpy="0 0 0" />
@@ -331,5 +338,5 @@
   <!-- ================================= -->
   <xacro:if value="$(arg use_sim)">
-    <gazebo reference="base_link">
+    <gazebo reference="chassis_link">
     </gazebo>
     <gazebo reference="camera_fisheye_yaw_link">
@@ -337,5 +344,7 @@
     <gazebo reference="front_right_wheel_link">
       <material>Gazebo/Grey</material>
-      <mu>1.0</mu>
+      <!-- Low friction along the axle (z in the collision frame) so skid turns can scrub -->
+      <fdir1>0 0 1</fdir1>
+      <mu1>0.3</mu1>
       <mu2>1.0</mu2>
       <surface>
@@ -352,5 +361,7 @@
     <gazebo reference="front_left_wheel_link">
       <material>Gazebo/Grey</material>
-      <mu>1.0</mu>
+      <!-- Low friction along the axle (z in the collision frame) so skid turns can scrub -->
+      <fdir1>0 0 1</fdir1>
+      <mu1>0.3</mu1>
       <mu2>1.0</mu2>
       <surface>
@@ -367,5 +378,7 @@
     <gazebo reference="rear_right_wheel_link">
       <material>Gazebo/Grey</material>
-      <mu>1.0</mu>
+      <!-- Low friction along the axle (z in the collision frame) so skid turns can scrub -->
+      <fdir1>0 0 1</fdir1>
+      <mu1>0.3</mu1>
       <mu2>1.0</mu2>
       <surface>
@@ -382,5 +395,7 @@
     <gazebo reference="rear_left_wheel_link">
       <material>Gazebo/Grey</material>
-      <mu>1.0</mu>
+      <!-- Low friction along the axle (z in the collision frame) so skid turns can scrub -->
+      <fdir1>0 0 1</fdir1>
+      <mu1>0.3</mu1>
       <mu2>1.0</mu2>
       <surface>
@@ -585,6 +600,6 @@
       <joint name="base_front_right_wheel_joint">
         <command_interface name="velocity">
-          <param name="min">-1</param>
-          <param name="max">1</param>
+          <param name="min">-5</param>
+          <param name="max">5</param>
         </command_interface>
         <state_interface name="position" />
@@ -593,6 +608,6 @@
       <joint name="base_front_left_wheel_joint">
         <command_interface name="velocity">
-          <param name="min">-1</param>
-          <param name="max">1</param>
+          <param name="min">-5</param>
+          <param name="max">5</param>
         </command_interface>
         <state_interface name="position" />
@@ -601,6 +616,6 @@
       <joint name="base_rear_right_wheel_joint">
         <command_interface name="velocity">
-          <param name="min">-1</param>
-          <param name="max">1</param>
+          <param name="min">-5</param>
+          <param name="max">5</param>
         </command_interface>
         <state_interface name="position" />
@@ -609,6 +624,6 @@
       <joint name="base_rear_left_wheel_joint">
         <command_interface name="velocity">
-          <param name="min">-1</param>
-          <param name="max">1</param>
+          <param name="min">-5</param>
+          <param name="max">5</param>
         </command_interface>
         <state_interface name="position" />
